File: LED_test.sch (KiCad schematic (older format))
At the start: 6 parts, among them J1 Conn_01x08_Male, J2 Conn_01x08_Male, U1 MAX14662

Commit message: Current PCB
Parts:
- removed J2: Conn_01x08_Male, Connector_PinHeader_2.00mm:PinHeader_1x08_P2.00mm_Vertical, symbol Connector:Conn_01x08_Male
- added J2: Conn_01x09_Male, Connector_PinHeader_2.00mm:PinHeader_1x09_P2.00mm_Vertical, symbol Connector:Conn_01x09_Male
Connections:
- net +12V: now also J2.5 (Pin_5)
- net +3V3: now also J2.7 (Pin_7)
- net +5V: now also J2.6 (Pin_6)
- net GND: now also J2.8 (Pin_8), J2.9 (Pin_9)
- net LED2/LED_Power: now also J2.1 (Pin_1)
- net LED2/SM_CLK: now also J2.2 (Pin_2)
- net LED2/SM_DATA: now also J2.3 (Pin_3)
- net Sheet5F1EB17F/DC_Current_Monitor: now also J2.4 (Pin_4)
Changed lines of the file:
@@
 	4650 2600 4300 2600
 Wire Wire Line
-	4650 2700 4300 2700
+	4650 2700 4400 2700
 $Comp
 L Device:R R2
@@
 	1    0    0    -1
 $EndComp
-$Comp
-L Connector:Conn_01x08_Male J2
-U 1 1 5F1D2EFD
-P 4100 2300
-F 0 "J2" H 4208 2781 50  0000 C CNN
-F 1 "Conn_01x08_Male" H 4208 2690 50  0000 C CNN
-F 2 "Connector_PinHeader_2.00mm:PinHeader_1x08_P2.00mm_Vertical" H 4100 2300 50  0001 C CNN
-F 3 "~" H 4100 2300 50  0001 C CNN
-	1    4100 2300
-	1    0    0    -1
-$EndComp
 Wire Wire Line
 	700  4150 2050 4150
@@
 	-1   0    0    1
 $EndComp
+$Comp
+L Connector:Conn_01x09_Male J2
+U 1 1 5F49C9B7
+P 4100 2400
+F 0 "J2" H 4208 2981 50  0000 C CNN
+F 1 "Conn_01x09_Male" H 4208 2890 50  0000 C CNN
+F 2 "Connector_PinHeader_2.00mm:PinHeader_1x09_P2.00mm_Vertical" H 4100 2400 50  0001 C CNN
+F 3 "~" H 4100 2400 50  0001 C CNN
+	1    4100 2400
+	1    0    0    -1
+$EndComp
+Wire Wire Line
+	4300 2800 4400 2800
+Wire Wire Line
+	4400 2800 4400 2700
+Connection ~ 4400 2700
+Wire Wire Line
+	4400 2700 4300 2700
 $EndSCHEMATC

Commit message: Current PCB
Parts:
- removed J2: Conn_01x09_Male, Connector_PinHeader_2.00mm:PinHeader_1x09_P2.00mm_Vertical, symbol Connector:Conn_01x09_Male
- added H1, H2, H3: MountingHole, MountingHole:MountingHole_3.5mm_Pad, symbol Mechanical:MountingHole
- added J2: Conn_01x14_Male, Connector_PinHeader_2.00mm:PinHeader_1x14_P2.00mm_Vertical, symbol Connector:Conn_01x14_Male
Connections:
- wire segments 70 -> 82
Other:
- moved on the sheet: C1, J1, R1, R2, U1
