File: LED_test.kicad_pcb (KiCad board)
At the start: 2 copper layers, 100 x 100 mm, 58 parts, among them J1 Conn_01x08_Male, J2 Conn_01x08_Male, Q1 FDC6330L, Q2 DMN6075S, U1 MAX14662, U2 MAX1978, U3 DAC081C085, U4 ADC101C021CIMM, U5 REF3333, U6 LTC1669CMS8, U7 AD8603, U8 PAC1931

Commit message: Current PCB
Parts:
- added R21: 0R, Resistor_SMD:R_0603_1608Metric_Pad1.05x0.95mm_HandSolder, F.Cu at (160.8, 119.6)
- added R22: 0R, Resistor_SMD:R_0603_1608Metric_Pad1.05x0.95mm_HandSolder, F.Cu at (166.4, 119.6)
- added R23: 0R, Resistor_SMD:R_0603_1608Metric_Pad1.05x0.95mm_HandSolder, F.Cu at (160.8, 124.7)
- added R24: 0R, Resistor_SMD:R_0603_1608Metric_Pad1.05x0.95mm_HandSolder, F.Cu at (166.4, 124.7)
- added R25: 0R, Resistor_SMD:R_0603_1608Metric_Pad1.05x0.95mm_HandSolder, F.Cu at (160.8, 129.0)
- added R26: 0R, Resistor_SMD:R_0603_1608Metric_Pad1.05x0.95mm_HandSolder, F.Cu at (166.4, 129.0)
- added R27: 0R, Resistor_SMD:R_0603_1608Metric_Pad1.05x0.95mm_HandSolder, F.Cu at (114.6, 50.5)
- added R28: 0R, Resistor_SMD:R_0603_1608Metric_Pad1.05x0.95mm_HandSolder, F.Cu at (118.9, 50.3)
- added R29: 0R, Resistor_SMD:R_0603_1608Metric_Pad1.05x0.95mm_HandSolder, F.Cu at (118.9, 45.5)
- added R30: 0R, Resistor_SMD:R_0603_1608Metric_Pad1.05x0.95mm_HandSolder, F.Cu at (114.8, 45.5)
- U6: value LTC1669CMS8 -> LTC1669IMS8
- moved C15 5.38 mm to (122.4, 54.6), turned to 0 degrees
- moved U6 3.97 mm to (174.0, 124.7)
Connections:
- U3 pad 1: (no net) -> Net-(R29-Pad2)
- U3 pad 2: (no net) -> Net-(R27-Pad2)
- U4 pad 3: (no net) -> Net-(R27-Pad2)
- U4 pad 6: (no net) -> Net-(R29-Pad2)
- U6 pad 2: GND -> Net-(R23-Pad1)
- U6 pad 3: GND -> Net-(R25-Pad1)
- U6 pad 6: GND -> Net-(R21-Pad1)
Routing:
- net +5V: track 471.7 -> 534.9 mm, vias 6 -> 8
- net Net-(R29-Pad2): track 0.00 -> 28.0 mm, vias 0 -> 3
- net Net-(R27-Pad2): track 0.00 -> 21.9 mm, vias 0 -> 2
- net Net-(R25-Pad1): track 0.00 -> 17.9 mm, vias 0 -> 2
- net Net-(R23-Pad1): track 0.00 -> 16.8 mm, vias 0 -> 2
- net Net-(R21-Pad1): track 0.00 -> 16.8 mm, vias 0 -> 2
- net Net-(U6-Pad8): track 23.6 -> 16.9 mm
- net /Sheet5F1EB17F/CLOCK: track 182.8 -> 186.6 mm
- net /Sheet5F1EB17F/DATA: track 199.1 -> 197.8 mm

Commit message: Current PCB
Routing:
- net Net-(R27-Pad2): track 21.9 -> 18.3 mm, vias 2 -> 0

Commit message: Current PCB
Parts:
- moved R7 0.93 mm to (137.2, 71.6), turned to 0 degrees
Routing:
- net Net-(C8-Pad1): track 37.9 -> 33.0 mm, vias 3 -> 2
- net VIN: track 40.8 -> 45.3 mm, vias 4 -> 2
- net Net-(C9-Pad2): track 3.26 -> 2.43 mm

Commit message: Current PCB
Parts:
- added C19: 1uF, Capacitor_SMD:C_0805_2012Metric_Pad1.15x1.40mm_HandSolder, F.Cu at (119.6, 63.5)
- added C20: 1uF, Capacitor_SMD:C_0805_2012Metric_Pad1.15x1.40mm_HandSolder, F.Cu at (126.5, 46.7)
- added C21: 4.7uF, Capacitor_Tantalum_SMD:CP_EIA-7343-15_Kemet-W_Pad2.25x2.55mm_HandSolder, F.Cu at (113.3, 46.5)
- added C22: 1uF, Capacitor_SMD:C_0805_2012Metric_Pad1.15x1.40mm_HandSolder, F.Cu at (112.8, 53.8)
- added C_PWR3: 100nF, Capacitor_SMD:C_0603_1608Metric_Pad1.05x0.95mm_HandSolder, F.Cu at (175.3, 119.1)
- added C_PWR4: 100nF, Capacitor_SMD:C_0603_1608Metric_Pad1.05x0.95mm_HandSolder, F.Cu at (179.8, 111.3)
- C18: value 100uF -> 4.7uF
- J2: value Conn_01x08_Male -> Conn_01x09_Male; footprint Connector_PinHeader_2.00mm:PinHeader_1x08_P2.00mm_Vertical -> Connector_PinHeader_2.00mm:PinHeader_1x09_P2.00mm_Vertical
- moved C18 55.9 mm to (122.2, 59.2)
- moved C16 32.8 mm to (139.7, 115.6), turned to 90 degrees
- moved R27 20.1 mm to (106.2, 68.8)
- moved R28 19.3 mm to (106.2, 64.8), turned to 270 degrees
- moved U5 17.5 mm to (131.1, 47.8)
- moved C15 14.7 mm to (133.1, 44.5)
- moved R29 14.2 mm to (105.7, 50.5), turned to 0 degrees
- moved R30 8.52 mm to (106.4, 47.0), turned to 270 degrees
- moved C4 8.18 mm to (129.0, 93.0)
- moved U4 7.89 mm to (108.7, 56.4)
- moved U3 7.12 mm to (113.3, 63.0)
- moved C_PWR2 5.40 mm to (186.4, 121.9), turned to 270 degrees
- moved C5 4.35 mm to (124.7, 95.2)
- moved R20 4.10 mm to (187.5, 99.8)
- moved C14 4.02 mm to (146.1, 89.2), turned to 270 degrees
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Connections:
- C18 pad 1: Net-(C18-Pad1) -> GND
- C18 pad 2: GND -> +5V
- D1 pad 2: Net-(C18-Pad1) -> Net-(D1-Pad2)
- Q1 pad 2: Net-(C18-Pad1) -> Net-(D1-Pad2)
- Q1 pad 3: Net-(C18-Pad1) -> Net-(D1-Pad2)
Routing:
- net /LED2/LED_Power: track 114.6 -> 62.5 mm, vias 4 -> 2
- net Net-(D1-Pad2): track 0.00 -> 50.1 mm
- net Net-(C18-Pad1): track 42.7 -> 0.00 mm
- net Net-(C20-Pad1): track 4.24 -> 26.5 mm, vias 0 -> 2
- net +5V: track 534.9 -> 551.7 mm, vias 8 -> 7
- net Net-(PE1-Pad1): track 33.4 -> 46.8 mm
- net Net-(R29-Pad2): track 28.0 -> 16.8 mm, vias 3 -> 0
- net VIN: track 45.3 -> 34.3 mm
- net GND: track 30.2 -> 19.4 mm, vias 7 -> 137
- net Net-(C12-Pad1): track 33.3 -> 40.7 mm
- net Net-(J1-Pad7): track 13.6 -> 6.78 mm
- net Net-(J1-Pad6): track 11.7 -> 5.86 mm
- net Net-(J1-Pad8): track 14.3 -> 8.62 mm
- net Net-(J1-Pad5): track 10.4 -> 5.19 mm
- net +3V3: track 118.3 -> 113.2 mm, vias 2 -> 1
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
Commit message: Current PCB
Parts:
- removed C21: 4.7uF, Capacitor_Tantalum_SMD:CP_EIA-7343-15_Kemet-W_Pad2.25x2.55mm_HandSolder
- added D1TH: PinHeader_1x02_P2.00mm_Vertical, Connector_PinHeader_2.00mm:PinHeader_1x02_P2.00mm_Vertical, F.Cu at (180.1, 86.6)
- added REF**: MountingHole_2.2mm_M2_DIN965_Pad, MountingHole:MountingHole_2.2mm_M2_DIN965_Pad, F.Cu at (196.1, 86.1)
- added REF**: MountingHole_2.2mm_M2_DIN965_Pad, MountingHole:MountingHole_2.2mm_M2_DIN965_Pad, F.Cu at (149.4, 43.2)
- added REF**: MountingHole_2.2mm_M2_DIN965_Pad, MountingHole:MountingHole_2.2mm_M2_DIN965_Pad, F.Cu at (102.9, 42.9)
- added REF**: MountingHole_2.2mm_M2_DIN965_Pad, MountingHole:MountingHole_2.2mm_M2_DIN965_Pad, F.Cu at (196.8, 136.9)
- added REF**: MountingHole_2.2mm_M2_DIN965_Pad, MountingHole:MountingHole_2.2mm_M2_DIN965_Pad, F.Cu at (102.6, 137.2)
- C18: footprint Capacitor_Tantalum_SMD:CP_EIA-7343-15_Kemet-W_Pad2.25x2.55mm_HandSolder -> Capacitor_SMD:C_0805_2012Metric_Pad1.15x1.40mm_HandSolder
- moved C16 31.7 mm to (169.9, 105.9), turned to 270 degrees
- moved R4 31.1 mm to (146.3, 77.0), turned to 270 degrees
- moved L1 29.8 mm to (135.4, 97.0)
- moved C14 24.5 mm to (154.2, 66.0), turned to 90 degrees
- moved R17 24.2 mm to (147.1, 79.5), turned to 0 degrees
- moved R5 23.7 mm to (144.8, 77.0), turned to 270 degrees
- moved R10 23.6 mm to (145.5, 83.6), turned to 90 degrees
- moved R3 23.4 mm to (139.4, 74.9), turned to 180 degrees
- moved C8 22.9 mm to (145.8, 88.1)
- moved L2 22.5 mm to (133.9, 64.8), turned to 0 degrees
- moved R7 18.4 mm to (142.7, 89.2), turned to 180 degrees
- moved R13 18.4 mm to (142.7, 82.5), turned to 0 degrees
- moved R8 18.2 mm to (114.0, 74.9)
- moved R9 18.0 mm to (117.6, 74.9)
- moved NTC1 17.2 mm to (149.1, 71.1), turned to 180 degrees
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Routing:
- net /Sheet5F1EB17F/DATA: track 201.4 -> 169.0 mm
- net +5V: track 551.7 -> 522.3 mm, vias 7 -> 13
- net /Sheet5F1EB17F/DC_Current_Monitor: track 72.1 -> 96.8 mm, vias 2 -> 1
- net Net-(PE1-Pad1): track 46.8 -> 70.7 mm
- net /Sheet5F1EB17F/CLOCK: track 187.3 -> 163.6 mm, vias 7 -> 4
- net Net-(U2-Pad19): track 28.9 -> 51.5 mm
- net Net-(NTC1-Pad1): track 43.4 -> 22.5 mm
- net REF: track 102.7 -> 84.0 mm
- net VIN: track 34.3 -> 52.7 mm
- net GND: track 19.4 -> 1.79 mm, vias 137 -> 88
- net Net-(C20-Pad1): track 26.5 -> 10.1 mm, vias 2 -> 0
- net Net-(D1-Pad2): track 50.1 -> 34.9 mm, vias 0 -> 160
- net Net-(C12-Pad1): track 40.7 -> 55.8 mm, vias 0 -> 2
- net Net-(C12-Pad2): track 38.2 -> 47.8 mm, vias 2 -> 0
- net Net-(C17-Pad2): track 63.7 -> 55.5 mm
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- added copper zone on B.Cu, net Net-(D1-Pad1)
- added copper zone on B.Cu, net Net-(D1-Pad2)
Other:
- rule trace_min: 0.2 -> 0.19

Commit message: Current PCB
Parts:
- removed D1TH: PinHeader_1x02_P2.00mm_Vertical, Connector_PinHeader_2.00mm:PinHeader_1x02_P2.00mm_Vertical
- removed REF** (x5): MountingHole_2.2mm_M2_DIN965_Pad, MountingHole:MountingHole_2.2mm_M2_DIN965_Pad
- added Extra_FP1: LED, Connector_PinHeader_2.00mm:PinHeader_1x02_P2.00mm_Vertical, F.Cu at (180.1, 86.1)
- added H1: MountingHole, MountingHole:MountingHole_3.5mm_Pad, F.Cu at (105.9, 133.8)
- added H2: MountingHole, MountingHole:MountingHole_3.5mm_Pad, F.Cu at (194.0, 134.5)
- added H3: MountingHole, MountingHole:MountingHole_3.5mm_Pad, F.Cu at (135.7, 46.9)
- C6, C7, R1, R2: moved to B.Cu
- J2: value Conn_01x09_Male -> Conn_01x14_Male; footprint Connector_PinHeader_2.00mm:PinHeader_1x09_P2.00mm_Vertical -> Connector_PinHeader_2.00mm:PinHeader_1x14_P2.00mm_Vertical
- moved R1 15.5 mm to (156.0, 131.1)
- moved C1 15.4 mm to (106.3, 112.9), turned to 270 degrees
- moved J1 12.3 mm to (113.3, 124.8), turned to 180 degrees
- moved R2 11.2 mm to (153.4, 132.3), turned to 270 degrees
- moved C7 8.82 mm to (124.0, 90.9)
- moved J2 8.30 mm to (120.9, 130.3), turned to 90 degrees
- moved U1 7.27 mm to (106.7, 118.1), turned to 0 degrees
- moved C6 4.18 mm to (130.2, 73.4)
- moved R_Address1 3.81 mm to (185.7, 131.8), turned to 180 degrees
- moved L1 2.84 mm to (135.9, 94.2), turned to 0 degrees
- moved C21 0.36 mm to (175.5, 118.9)
- renumbered C_PWR3 to C21, C_PWR4 to C23, C_PWR1 to C24, C_PWR2 to C25
Connections:
- J2 pad 1: /LED2/LED_Power -> GND
- J2 pad 3: /Sheet5F1EB17F/DATA -> GND
- J2 pad 4: /Sheet5F1EB17F/DC_Current_Monitor -> /Sheet5F1EB17F/DATA
- J2 pad 5: +12V -> GND
- J2 pad 6: +5V -> /Sheet5F1EB17F/DC_Current_Monitor
- J2 pad 7: +3V3 -> /LED2/LED_Power
- J2 pad 9: GND -> +12V
Routing:
- net +5V: track 522.3 -> 450.8 mm, vias 13 -> 8
- net +3V3: track 106.1 -> 71.3 mm, vias 3 -> 1
- net Net-(L2-Pad1): track 43.1 -> 23.4 mm
- net +12V: track 76.4 -> 58.2 mm, vias 1 -> 0
- net Net-(L1-Pad1): track 32.2 -> 16.2 mm
- net /LED2/LED_Power: track 67.2 -> 61.0 mm
- net /Sheet5F1EB17F/DATA: track 169.0 -> 175.1 mm, vias 0 -> 3
- net /Sheet5F1EB17F/CLOCK: track 163.6 -> 166.7 mm, vias 4 -> 1
- net GND: track 1.79 -> 0.02 mm, vias 88 -> 99
- net Net-(C12-Pad2): track 47.8 -> 49.3 mm
- net Net-(R_Address1-Pad1): track 3.21 -> 2.30 mm
- net Net-(R10-Pad2): track 11.7 -> 11.0 mm
- net /Sheet5F1EB17F/DC_Current_Monitor: track 96.8 -> 96.7 mm, vias 1 -> 0

Commit message: Current PCB
Parts:
- U2: footprint Package_DFN_QFN:QFN-48-1EP_7x7mm_P0.5mm_EP5.45x5.45mm -> Package_DFN_QFN:QFN-48-1EP_7x7mm_P0.5mm_EP5.45x5.45mm_ThermalVias
Connections:
- U2 pad 49: (no net) -> GND
Routing:
- net GND: track 0.02 -> 32.5 mm
