File: Peltier_V2.sch (KiCad schematic (older format))
At the start: 37 parts, among them U2 MAX1978, U3 DAC081C085, U4 ADC101C021CIMM, U5 REF3333

Commit message: Current PCB
Parts:
- added R27, R28, R29, R30: 0R, Resistor_SMD:R_0603_1608Metric_Pad1.05x0.95mm_HandSolder, symbol Device:R
Connections:
- wire segments 163 -> 181
Other:
- note added: "These two IC follow same \naddressing schematics,\n can be connected together"
- moved on the sheet: U4
Changed lines of the file:
@@
 L Analog_ADC:ADC101C021CIMM U?
 U 1 1 5F2DF3E0
-P 8550 3950
+P 9550 3550
 AR Path="/5F115F8B/5F2DF3E0" Ref="U?"  Part="1"
 AR Path="/5F1EB180/5F2DF3E0" Ref="U4"  Part="1"
 AR Path="/5F22BCD9/5F22EBB8/5F2DF3E0" Ref="U?"  Part="1"
-F 0 "U4" H 8350 4200 31  0000 C CNN
-F 1 "ADC101C021CIMM" H 8850 4200 31  0000 C CNN
-F 2 "Package_SO:MSOP-8_3x3mm_P0.65mm" H 9350 3600 50  0001 C CNN
-F 3 "http://www.ti.com/lit/ds/symlink/adc101c021.pdf" H 8550 4050 50  0001 C CNN
-	1    8550 3950
+F 0 "U4" H 9350 3800 31  0000 C CNN
+F 1 "ADC101C021CIMM" H 9850 3800 31  0000 C CNN
+F 2 "Package_SO:MSOP-8_3x3mm_P0.65mm" H 10350 3200 50  0001 C CNN
+F 3 "http://www.ti.com/lit/ds/symlink/adc101c021.pdf" H 9550 3650 50  0001 C CNN
+	1    9550 3550
 	1    0    0    -1
 $EndComp
@@
 L power:+5V #PWR019
 U 1 1 5F2F73EE
-P 8550 3450
+P 9550 3050
 AR Path="/5F1EB180/5F2F73EE" Ref="#PWR019"  Part="1"
 AR Path="/5F22BCD9/5F22EBB8/5F2F73EE" Ref="#PWR?"  Part="1"
-F 0 "#PWR019" H 8550 3300 50  0001 C CNN
-F 1 "+5V" H 8565 3623 50  0000 C CNN
-F 2 "" H 8550 3450 50  0001 C CNN
-F 3 "" H 8550 3450 50  0001 C CNN
-	1    8550 3450
+F 0 "#PWR019" H 9550 2900 50  0001 C CNN
+F 1 "+5V" H 9565 3223 50  0000 C CNN
+F 2 "" H 9550 3050 50  0001 C CNN
+F 3 "" H 9550 3050 50  0001 C CNN
+	1    9550 3050
 	1    0    0    -1
 $EndComp
@@
 L power:GND #PWR020
 U 1 1 5F2F78D2
-P 8550 4350
+P 9550 3950
 AR Path="/5F1EB180/5F2F78D2" Ref="#PWR020"  Part="1"
 AR Path="/5F22BCD9/5F22EBB8/5F2F78D2" Ref="#PWR?"  Part="1"
-F 0 "#PWR020" H 8550 4100 50  0001 C CNN
-F 1 "GND" H 8555 4177 50  0000 C CNN
-F 2 "" H 8550 4350 50  0001 C CNN
-F 3 "" H 8550 4350 50  0001 C CNN
-	1    8550 4350
+F 0 "#PWR020" H 9550 3700 50  0001 C CNN
+F 1 "GND" H 9555 3777 50  0000 C CNN
+F 2 "" H 9550 3950 50  0001 C CNN
+F 3 "" H 9550 3950 50  0001 C CNN
+	1    9550 3950
 	1    0    0    -1
 $EndComp
 Wire Wire Line
-	8550 3450 8550 3650
-Wire Wire Line
-	8550 4250 8550 4350
+	9550 3050 9550 3250
+Wire Wire Line
+	9550 3850 9550 3950
 Wire Wire Line
 	1150 4150 1700 4150
 Text GLabel 1150 4150 0    50   BiDi ~ 0
 VIN
-Text GLabel 7950 3800 1    50   BiDi ~ 0
+Text GLabel 8950 3400 1    50   BiDi ~ 0
 VIN
 Wire Wire Line
-	7950 3850 7950 3800
-Wire Wire Line
-	7950 3850 8150 3850
-Text HLabel 9450 3850 2    50   BiDi ~ 0
+	8950 3450 8950 3400
+Wire Wire Line
+	8950 3450 9150 3450
+Text HLabel 10450 3450 2    50   BiDi ~ 0
 CLOCK
-Text HLabel 9450 3950 2    50   BiDi ~ 0
+Text HLabel 10450 3550 2    50   BiDi ~ 0
 DATA
 Wire Wire Line
-	8950 3850 9050 3850
-Wire Wire Line
-	9450 3950 9150 3950
-Wire Wire Line
-	8050 5250 9050 5250
-Wire Wire Line
-	9050 5250 9050 3850
-Connection ~ 9050 3850
-Wire Wire Line
-	9050 3850 9450 3850
-Wire Wire Line
-	8050 5350 9150 5350
-Wire Wire Line
-	9150 5350 9150 3950
-Connection ~ 9150 3950
-Wire Wire Line
-	9150 3950 8950 3950
+	9950 3450 10050 3450
+Wire Wire Line
+	10450 3550 10150 3550
+Connection ~ 10050 3450
+Wire Wire Line
+	10050 3450 10450 3450
+Connection ~ 10150 3550
+Wire Wire Line
+	10150 3550 9950 3550
 $Comp
 L power:GND #PWR013
@@
 	2900 5050 3150 5050
 Connection ~ 3150 5050
+$Comp
+L Device:R R27
+U 1 1 5F3C7569
+P 8350 3550
+AR Path="/5F1EB180/5F3C7569" Ref="R27"  Part="1"
+AR Path="/5F22BCD9/5F22EBB8/5F3C7569" Ref="R?"  Part="1"
+F 0 "R27" H 8420 3596 50  0000 L CNN
+F 1 "0R" V 8350 3500 50  0000 L CNN
+F 2 "Resistor_SMD:R_0603_1608Metric_Pad1.05x0.95mm_HandSolder" V 8280 3550 50  0001 C CNN
+F 3 "~" H 8350 3550 50  0001 C CNN
+	1    8350 3550
+	0    -1   -1   0
+$EndComp
+Wire Wire Line
+	10050 3450 10050 5250
+Wire Wire Line
+	8050 5250 10050 5250
+Wire Wire Line
+	8050 5350 10150 5350
+Wire Wire Line
+	10150 3550 10150 5350
+$Comp
+L Device:R R28
+U 1 1 5F3E943D
+P 8350 3800
+AR Path="/5F1EB180/5F3E943D" Ref="R28"  Part="1"
+AR Path="/5F22BCD9/5F22EBB8/5F3E943D" Ref="R?"  Part="1"
+F 0 "R28" H 8420 3846 50  0000 L CNN
+F 1 "0R" V 8350 3750 50  0000 L CNN
+F 2 "Resistor_SMD:R_0603_1608Metric_Pad1.05x0.95mm_HandSolder" V 8280 3800 50  0001 C CNN
+F 3 "~" H 8350 3800 50  0001 C CNN
+	1    8350 3800
+	0    -1   -1   0
+$EndComp
+$Comp
+L Device:R R29
+U 1 1 5F3E9805
+P 8350 4050
+AR Path="/5F1EB180/5F3E9805" Ref="R29"  Part="1"
+AR Path="/5F22BCD9/5F22EBB8/5F3E9805" Ref="R?"  Part="1"
+F 0 "R29" H 8420 4096 50  0000 L CNN
+F 1 "0R" V 8350 4000 50  0000 L CNN
+F 2 "Resistor_SMD:R_0603_1608Metric_Pad1.05x0.95mm_HandSolder" V 8280 4050 50  0001 C CNN
+F 3 "~" H 8350 4050 50  0001 C CNN
+	1    8350 4050
+	0    -1   -1   0
+$EndComp
+$Comp
+L Device:R R30
+U 1 1 5F3E9A55
+P 8350 4350
+AR Path="/5F1EB180/5F3E9A55" Ref="R30"  Part="1"
+AR Path="/5F22BCD9/5F22EBB8/5F3E9A55" Ref="R?"  Part="1"
+F 0 "R30" H 8420 4396 50  0000 L CNN
+F 1 "0R" V 8350 4300 50  0000 L CNN
+F 2 "Resistor_SMD:R_0603_1608Metric_Pad1.05x0.95mm_HandSolder" V 8280 4350 50  0001 C CNN
+F 3 "~" H 8350 4350 50  0001 C CNN
+	1    8350 4350
+	0    -1   -1   0
+$EndComp
+$Comp
+L power:+5V #PWR035
+U 1 1 5F3F28AE
+P 8050 3550
+AR Path="/5F1EB180/5F3F28AE" Ref="#PWR035"  Part="1"
+AR Path="/5F22BCD9/5F22EBB8/5F3F28AE" Ref="#PWR?"  Part="1"
+F 0 "#PWR035" H 8050 3400 50  0001 C CNN
+F 1 "+5V" H 8065 3723 50  0000 C CNN
+F 2 "" H 8050 3550 50  0001 C CNN
+F 3 "" H 8050 3550 50  0001 C CNN
+	1    8050 3550
+	0    -1   -1   0
+$EndComp
+$Comp
+L power:GND #PWR036
+U 1 1 5F41126E
+P 8050 3800
+AR Path="/5F1EB180/5F41126E" Ref="#PWR036"  Part="1"
+AR Path="/5F22BCD9/5F22EBB8/5F41126E" Ref="#PWR?"  Part="1"
+F 0 "#PWR036" H 8050 3550 50  0001 C CNN
+F 1 "GND" H 8055 3627 50  0000 C CNN
+F 2 "" H 8050 3800 50  0001 C CNN
+F 3 "" H 8050 3800 50  0001 C CNN
+	1    8050 3800
+	0    1    1    0
+$EndComp
+Wire Wire Line
+	8050 3550 8150 3550
+Wire Wire Line
+	8500 3550 8700 3550
+Wire Wire Line
+	8500 3550 8500 3800
+Connection ~ 8500 3550
+Wire Wire Line
+	8200 3800 8050 3800
+Wire Wire Line
+	8200 4050 8150 4050
+Wire Wire Line
+	8150 4050 8150 3550
+Connection ~ 8150 3550
+Wire Wire Line
+	8150 3550 8200 3550
+Wire Wire Line
+	8050 3800 8050 4350
+Wire Wire Line
+	8050 4350 8200 4350
+Connection ~ 8050 3800
+Wire Wire Line
+	9150 3650 8600 3650
+Wire Wire Line
+	8600 3650 8600 4050
+Wire Wire Line
+	8600 4050 8500 4050
+Wire Wire Line
+	8500 4050 8500 4350
+Connection ~ 8500 4050
+Wire Wire Line
+	8050 4900 8500 4900
+Wire Wire Line
+	8500 4900 8500 4350
+Connection ~ 8500 4350
+Wire Wire Line
+	8050 5000 8700 5000
+Wire Wire Line
+	8700 5000 8700 3550
+Connection ~ 8700 3550
+Wire Wire Line
+	8700 3550 9150 3550
+Text Notes 9050 4700 0    39   ~ 0
+These two IC follow same \naddressing schematics,\n can be connected together
+Wire Notes Line
+	9350 3950 9350 4450
+Wire Notes Line
+	8400 5100 9350 5100
+Wire Notes Line
+	9350 5100 9350 4750
+Wire Notes Line
+	9300 4000 9350 3950
+Wire Notes Line
+	9350 3950 9400 4000
+Wire Notes Line
+	8400 5100 8450 5050
+Wire Notes Line
+	8400 5100 8450 5150
 $EndSCHEMATC

Commit message: Current PCB
Parts:
- added C18, C21: 4.7uF, Capacitor_Tantalum_SMD:CP_EIA-7343-15_Kemet-W_Pad2.25x2.55mm_HandSolder, symbol Device:CP
- added C19, C20, C22: 1uF, Capacitor_SMD:C_0805_2012Metric_Pad1.15x1.40mm_HandSolder, symbol Device:C
Connections:
- wire segments 181 -> 200
Changed lines of the file:
@@
 L power:+5V #PWR018
 U 1 1 5F2D255B
-P 7700 4600
+P 7700 4250
 AR Path="/5F1EB180/5F2D255B" Ref="#PWR018"  Part="1"
 AR Path="/5F22BCD9/5F22EBB8/5F2D255B" Ref="#PWR?"  Part="1"
-F 0 "#PWR018" H 7700 4450 50  0001 C CNN
-F 1 "+5V" H 7715 4773 50  0000 C CNN
-F 2 "" H 7700 4600 50  0001 C CNN
-F 3 "" H 7700 4600 50  0001 C CNN
-	1    7700 4600
-	1    0    0    -1
-$EndComp
-Wire Wire Line
-	7700 4600 7700 4700
+F 0 "#PWR018" H 7700 4100 50  0001 C CNN
+F 1 "+5V" H 7715 4423 50  0000 C CNN
+F 2 "" H 7700 4250 50  0001 C CNN
+F 3 "" H 7700 4250 50  0001 C CNN
+	1    7700 4250
+	1    0    0    -1
+$EndComp
+Wire Wire Line
+	7700 4250 7700 4300
 $Comp
 L Analog_ADC:ADC101C021CIMM U?
@@
 AR Path="/5F1EB180/5F2DF3E0" Ref="U4"  Part="1"
 AR Path="/5F22BCD9/5F22EBB8/5F2DF3E0" Ref="U?"  Part="1"
-F 0 "U4" H 9350 3800 31  0000 C CNN
+F 0 "U4" H 9450 3700 31  0000 C CNN
 F 1 "ADC101C021CIMM" H 9850 3800 31  0000 C CNN
 F 2 "Package_SO:MSOP-8_3x3mm_P0.65mm" H 10350 3200 50  0001 C CNN
@@
 L power:+5V #PWR019
 U 1 1 5F2F73EE
-P 9550 3050
+P 9550 2150
 AR Path="/5F1EB180/5F2F73EE" Ref="#PWR019"  Part="1"
 AR Path="/5F22BCD9/5F22EBB8/5F2F73EE" Ref="#PWR?"  Part="1"
-F 0 "#PWR019" H 9550 2900 50  0001 C CNN
-F 1 "+5V" H 9565 3223 50  0000 C CNN
-F 2 "" H 9550 3050 50  0001 C CNN
-F 3 "" H 9550 3050 50  0001 C CNN
-	1    9550 3050
+F 0 "#PWR019" H 9550 2000 50  0001 C CNN
+F 1 "+5V" H 9565 2323 50  0000 C CNN
+F 2 "" H 9550 2150 50  0001 C CNN
+F 3 "" H 9550 2150 50  0001 C CNN
+	1    9550 2150
 	1    0    0    -1
 $EndComp
@@
 $EndComp
 Wire Wire Line
-	9550 3050 9550 3250
+	9550 2150 9550 2500
 Wire Wire Line
 	9550 3850 9550 3950
@@
 	8050 5450 8550 5450
 Wire Wire Line
-	6850 6250 8950 6250
+	6850 6250 8200 6250
 Connection ~ 6850 6250
 Wire Wire Line
@@
 Wire Notes Line
 	8400 5100 8450 5150
+$Comp
+L Device:C C20
+U 1 1 5F34CB68
+P 8350 5800
+AR Path="/5F1EB180/5F34CB68" Ref="C20"  Part="1"
+AR Path="/5F22BCD9/5F22EBB8/5F34CB68" Ref="C?"  Part="1"
+F 0 "C20" H 8465 5846 50  0000 L CNN
+F 1 "1uF" H 8465 5755 50  0000 L CNN
+F 2 "Capacitor_SMD:C_0805_2012Metric_Pad1.15x1.40mm_HandSolder" H 8388 5650 50  0001 C CNN
+F 3 "~" H 8350 5800 50  0001 C CNN
+	1    8350 5800
+	0    1    1    0
+$EndComp
+Wire Wire Line
+	8500 5800 8550 5800
+Connection ~ 8550 5800
+Wire Wire Line
+	8200 5800 8200 6250
+Connection ~ 8200 6250
+Wire Wire Line
+	8200 6250 8950 6250
+$Comp
+L Device:C C19
+U 1 1 5F35F47B
+P 7350 4600
+AR Path="/5F1EB180/5F35F47B" Ref="C19"  Part="1"
+AR Path="/5F22BCD9/5F22EBB8/5F35F47B" Ref="C?"  Part="1"
+F 0 "C19" H 7465 4646 50  0000 L CNN
+F 1 "1uF" H 7465 4555 50  0000 L CNN
+F 2 "Capacitor_SMD:C_0805_2012Metric_Pad1.15x1.40mm_HandSolder" H 7388 4450 50  0001 C CNN
+F 3 "~" H 7350 4600 50  0001 C CNN
+	1    7350 4600
+	0    1    1    0
+$EndComp
+$Comp
+L power:GND #PWR027
+U 1 1 5F360708
+P 7150 4600
+AR Path="/5F1EB180/5F360708" Ref="#PWR027"  Part="1"
+AR Path="/5F22BCD9/5F22EBB8/5F360708" Ref="#PWR?"  Part="1"
+F 0 "#PWR027" H 7150 4350 50  0001 C CNN
+F 1 "GND" H 7155 4427 50  0000 C CNN
+F 2 "" H 7150 4600 50  0001 C CNN
+F 3 "" H 7150 4600 50  0001 C CNN
+	1    7150 4600
+	1    0    0    -1
+$EndComp
+Wire Wire Line
+	7150 4600 7200 4600
+Wire Wire Line
+	7500 4600 7700 4600
+Connection ~ 7700 4600
+Wire Wire Line
+	7700 4600 7700 4700
+Wire Wire Line
+	7450 4200 7600 4200
+Wire Wire Line
+	7600 4200 7600 4300
+Wire Wire Line
+	7600 4300 7700 4300
+Connection ~ 7700 4300
+Wire Wire Line
+	7700 4300 7700 4600
+Wire Wire Line
+	7150 4200 7150 4600
+Connection ~ 7150 4600
+$Comp
+L Device:CP C18
+U 1 1 5F40B4CF
+P 7300 4200
+AR Path="/5F1EB180/5F40B4CF" Ref="C18"  Part="1"
+AR Path="/5F22BCD9/5F22EBB8/5F40B4CF" Ref="C?"  Part="1"
+F 0 "C18" V 7555 4200 50  0000 C CNN
+F 1 "4.7uF" V 7464 4200 50  0000 C CNN
+F 2 "Capacitor_Tantalum_SMD:CP_EIA-7343-15_Kemet-W_Pad2.25x2.55mm_HandSolder" H 7338 4050 50  0001 C CNN
+F 3 "~" H 7300 4200 50  0001 C CNN
+	1    7300 4200
+	0    -1   -1   0
+$EndComp
+$Comp
+L Device:C C22
+U 1 1 5F419CCE
+P 9250 2900
+AR Path="/5F1EB180/5F419CCE" Ref="C22"  Part="1"
+AR Path="/5F22BCD9/5F22EBB8/5F419CCE" Ref="C?"  Part="1"
+F 0 "C22" H 9365 2946 50  0000 L CNN
+F 1 "1uF" H 9365 2855 50  0000 L CNN
+F 2 "Capacitor_SMD:C_0805_2012Metric_Pad1.15x1.40mm_HandSolder" H 9288 2750 50  0001 C CNN
+F 3 "~" H 9250 2900 50  0001 C CNN
+	1    9250 2900
+	0    1    1    0
+$EndComp
+$Comp
+L power:GND #PWR028
+U 1 1 5F419CD4
+P 9000 2700
+AR Path="/5F1EB180/5F419CD4" Ref="#PWR028"  Part="1"
+AR Path="/5F22BCD9/5F22EBB8/5F419CD4" Ref="#PWR?"  Part="1"
+F 0 "#PWR028" H 9000 2450 50  0001 C CNN
+F 1 "GND" H 9005 2527 50  0000 C CNN
+F 2 "" H 9000 2700 50  0001 C CNN
+F 3 "" H 9000 2700 50  0001 C CNN
+	1    9000 2700
+	0    1    1    0
+$EndComp
+$Comp
+L Device:CP C21
+U 1 1 5F419CDD
+P 9200 2500
+AR Path="/5F1EB180/5F419CDD" Ref="C21"  Part="1"
+AR Path="/5F22BCD9/5F22EBB8/5F419CDD" Ref="C?"  Part="1"
+F 0 "C21" V 9455 2500 50  0000 C CNN
+F 1 "4.7uF" V 9364 2500 50  0000 C CNN
+F 2 "Capacitor_Tantalum_SMD:CP_EIA-7343-15_Kemet-W_Pad2.25x2.55mm_HandSolder" H 9238 2350 50  0001 C CNN
+F 3 "~" H 9200 2500 50  0001 C CNN
+	1    9200 2500
+	0    -1   -1   0
+$EndComp
+Wire Wire Line
+	9350 2500 9550 2500
+Connection ~ 9550 2500
+Wire Wire Line
+	9550 2500 9550 2900
+Wire Wire Line
+	9400 2900 9550 2900
+Connection ~ 9550 2900
+Wire Wire Line
+	9550 2900 9550 3250
+Wire Wire Line
+	9000 2900 9000 2700
+Wire Wire Line
+	9000 2900 9100 2900
+Wire Wire Line
+	9000 2700 9000 2500
+Wire Wire Line
+	9000 2500 9050 2500
+Connection ~ 9000 2700
 $EndSCHEMATC

Commit message: Current PCB
Parts:
- removed C18, C21: 4.7uF, Capacitor_Tantalum_SMD:CP_EIA-7343-15_Kemet-W_Pad2.25x2.55mm_HandSolder, symbol Device:CP
- added C18: 4.7uF, Capacitor_SMD:C_0805_2012Metric_Pad1.15x1.40mm_HandSolder, symbol Device:C
Connections:
- wire segments 200 -> 195
Changed lines of the file:
@@
 	1    0    0    -1
 $EndComp
-Wire Wire Line
-	7700 4250 7700 4300
 $Comp
 L Analog_ADC:ADC101C021CIMM U?
@@
 Wire Wire Line
 	7700 4600 7700 4700
-Wire Wire Line
-	7450 4200 7600 4200
-Wire Wire Line
-	7600 4200 7600 4300
-Wire Wire Line
-	7600 4300 7700 4300
-Connection ~ 7700 4300
-Wire Wire Line
-	7700 4300 7700 4600
-Wire Wire Line
-	7150 4200 7150 4600
-Connection ~ 7150 4600
-$Comp
-L Device:CP C18
-U 1 1 5F40B4CF
-P 7300 4200
-AR Path="/5F1EB180/5F40B4CF" Ref="C18"  Part="1"
-AR Path="/5F22BCD9/5F22EBB8/5F40B4CF" Ref="C?"  Part="1"
-F 0 "C18" V 7555 4200 50  0000 C CNN
-F 1 "4.7uF" V 7464 4200 50  0000 C CNN
-F 2 "Capacitor_Tantalum_SMD:CP_EIA-7343-15_Kemet-W_Pad2.25x2.55mm_HandSolder" H 7338 4050 50  0001 C CNN
-F 3 "~" H 7300 4200 50  0001 C CNN
-	1    7300 4200
-	0    -1   -1   0
-$EndComp
 $Comp
 L Device:C C22
@@
 	0    1    1    0
 $EndComp
-$Comp
-L Device:CP C21
-U 1 1 5F419CDD
+Wire Wire Line
+	9350 2500 9550 2500
+Connection ~ 9550 2500
+Wire Wire Line
+	9550 2500 9550 2900
+Wire Wire Line
+	9400 2900 9550 2900
+Connection ~ 9550 2900
+Wire Wire Line
+	9550 2900 9550 3250
+Wire Wire Line
+	9000 2900 9000 2700
+Wire Wire Line
+	9000 2900 9100 2900
+Wire Wire Line
+	9000 2700 9000 2500
+Wire Wire Line
+	9000 2500 9050 2500
+Connection ~ 9000 2700
+$Comp
+L Device:C C18
+U 1 1 5F359FA4
 P 9200 2500
-AR Path="/5F1EB180/5F419CDD" Ref="C21"  Part="1"
-AR Path="/5F22BCD9/5F22EBB8/5F419CDD" Ref="C?"  Part="1"
-F 0 "C21" V 9455 2500 50  0000 C CNN
-F 1 "4.7uF" V 9364 2500 50  0000 C CNN
-F 2 "Capacitor_Tantalum_SMD:CP_EIA-7343-15_Kemet-W_Pad2.25x2.55mm_HandSolder" H 9238 2350 50  0001 C CNN
+AR Path="/5F1EB180/5F359FA4" Ref="C18"  Part="1"
+AR Path="/5F22BCD9/5F22EBB8/5F359FA4" Ref="C?"  Part="1"
+F 0 "C18" H 9315 2546 50  0000 L CNN
+F 1 "4.7uF" H 9315 2455 50  0000 L CNN
+F 2 "Capacitor_SMD:C_0805_2012Metric_Pad1.15x1.40mm_HandSolder" H 9238 2350 50  0001 C CNN
 F 3 "~" H 9200 2500 50  0001 C CNN
 	1    9200 2500
@@
 $EndComp
 Wire Wire Line
-	9350 2500 9550 2500
-Connection ~ 9550 2500
-Wire Wire Line
-	9550 2500 9550 2900
-Wire Wire Line
-	9400 2900 9550 2900
-Connection ~ 9550 2900
-Wire Wire Line
-	9550 2900 9550 3250
-Wire Wire Line
-	9000 2900 9000 2700
-Wire Wire Line
-	9000 2900 9100 2900
-Wire Wire Line
-	9000 2700 9000 2500
-Wire Wire Line
-	9000 2500 9050 2500
-Connection ~ 9000 2700
+	7700 4250 7700 4600
 $EndSCHEMATC

Commit message: Current PCB
Connections:
- wire segments 195 -> 198
Changed lines of the file:
@@
 Wire Wire Line
 	5000 1800 5000 1850
-$Comp
-L Device:R R?
-U 1 1 5F1FFA29
-P 5000 1650
-AR Path="/5F115F8B/5F1FFA29" Ref="R?"  Part="1"
-AR Path="/5F1EB180/5F1FFA29" Ref="R8"  Part="1"
-AR Path="/5F22BCD9/5F22EBB8/5F1FFA29" Ref="R?"  Part="1"
-F 0 "R8" H 4850 1800 50  0000 L CNN
-F 1 "R" V 5000 1600 50  0000 L CNN
-F 2 "Resistor_SMD:R_0603_1608Metric_Pad1.05x0.95mm_HandSolder" V 4930 1650 50  0001 C CNN
-F 3 "~" H 5000 1650 50  0001 C CNN
-	1    5000 1650
-	1    0    0    -1
-$EndComp
-$Comp
-L Device:R R?
-U 1 1 5F1FFA23
-P 5000 2050
-AR Path="/5F115F8B/5F1FFA23" Ref="R?"  Part="1"
-AR Path="/5F1EB180/5F1FFA23" Ref="R9"  Part="1"
-AR Path="/5F22BCD9/5F22EBB8/5F1FFA23" Ref="R?"  Part="1"
-F 0 "R9" H 5000 2200 50  0000 L CNN
-F 1 "R" V 5000 2000 50  0000 L CNN
-F 2 "Resistor_SMD:R_0603_1608Metric_Pad1.05x0.95mm_HandSolder" V 4930 2050 50  0001 C CNN
-F 3 "~" H 5000 2050 50  0001 C CNN
-	1    5000 2050
-	1    0    0    -1
-$EndComp
 Wire Wire Line
 	5450 1850 5450 1900
@@
 	5200 1500 5200 1350
 $Comp
-L Device:R R?
-U 1 1 5F1FFA16
-P 5450 1650
-AR Path="/5F115F8B/5F1FFA16" Ref="R?"  Part="1"
-AR Path="/5F1EB180/5F1FFA16" Ref="R14"  Part="1"
-AR Path="/5F22BCD9/5F22EBB8/5F1FFA16" Ref="R?"  Part="1"
-F 0 "R14" H 5450 1800 50  0000 L CNN
-F 1 "R" V 5450 1600 50  0000 L CNN
-F 2 "Resistor_SMD:R_0603_1608Metric_Pad1.05x0.95mm_HandSolder" V 5380 1650 50  0001 C CNN
-F 3 "~" H 5450 1650 50  0001 C CNN
-	1    5450 1650
-	1    0    0    -1
-$EndComp
-$Comp
-L Device:R R?
-U 1 1 5F1FFA10
-P 5200 1650
-AR Path="/5F115F8B/5F1FFA10" Ref="R?"  Part="1"
-AR Path="/5F1EB180/5F1FFA10" Ref="R11"  Part="1"
-AR Path="/5F22BCD9/5F22EBB8/5F1FFA10" Ref="R?"  Part="1"
-F 0 "R11" H 5200 1800 50  0000 L CNN
-F 1 "R" V 5200 1600 50  0000 L CNN
-F 2 "Resistor_SMD:R_0603_1608Metric_Pad1.05x0.95mm_HandSolder" V 5130 1650 50  0001 C CNN
-F 3 "~" H 5200 1650 50  0001 C CNN
-	1    5200 1650
-	1    0    0    -1
-$EndComp
-$Comp
-L Device:R R?
-U 1 1 5F1FFA0A
-P 5450 2050
-AR Path="/5F115F8B/5F1FFA0A" Ref="R?"  Part="1"
-AR Path="/5F1EB180/5F1FFA0A" Ref="R15"  Part="1"
-AR Path="/5F22BCD9/5F22EBB8/5F1FFA0A" Ref="R?"  Part="1"
-F 0 "R15" H 5450 2200 50  0000 L CNN
-F 1 "R" V 5450 2000 50  0000 L CNN
-F 2 "Resistor_SMD:R_0603_1608Metric_Pad1.05x0.95mm_HandSolder" V 5380 2050 50  0001 C CNN
-F 3 "~" H 5450 2050 50  0001 C CNN
-	1    5450 2050
-	1    0    0    -1
-$EndComp
-$Comp
-L Device:R R?
-U 1 1 5F1FFA04
-P 5200 2050
-AR Path="/5F115F8B/5F1FFA04" Ref="R?"  Part="1"
-AR Path="/5F1EB180/5F1FFA04" Ref="R12"  Part="1"
-AR Path="/5F22BCD9/5F22EBB8/5F1FFA04" Ref="R?"  Part="1"
-F 0 "R12" H 5200 2200 50  0000 L CNN
-F 1 "R" V 5200 2000 50  0000 L CNN
-F 2 "Resistor_SMD:R_0603_1608Metric_Pad1.05x0.95mm_HandSolder" V 5130 2050 50  0001 C CNN
-F 3 "~" H 5200 2050 50  0001 C CNN
-	1    5200 2050
-	1    0    0    -1
-$EndComp
-$Comp
 L power:GND #PWR?
 U 1 1 5F1FF9FE
-P 5200 1350
+P 5850 2100
 AR Path="/5F0387D4/5F1FF9FE" Ref="#PWR?"  Part="1"
 AR Path="/5F115F8B/5F1FF9FE" Ref="#PWR?"  Part="1"
 AR Path="/5F1EB180/5F1FF9FE" Ref="#PWR014"  Part="1"
 AR Path="/5F22BCD9/5F22EBB8/5F1FF9FE" Ref="#PWR?"  Part="1"
-F 0 "#PWR014" H 5200 1100 50  0001 C CNN
-F 1 "GND" H 5205 1177 50  0000 C CNN
-F 2 "" H 5200 1350 50  0001 C CNN
-F 3 "" H 5200 1350 50  0001 C CNN
-	1    5200 1350
-	-1   0    0    1
+F 0 "#PWR014" H 5850 1850 50  0001 C CNN
+F 1 "GND" H 5855 1927 50  0000 C CNN
+F 2 "" H 5850 2100 50  0001 C CNN
+F 3 "" H 5850 2100 50  0001 C CNN
+	1    5850 2100
+	1    0    0    -1
 $EndComp
 Wire Wire Line
@@
 $EndComp
 Connection ~ 4200 1850
-Wire Wire Line
-	4200 1250 4200 1450
 Wire Wire Line
 	3850 1850 4200 1850
@@
 L power:GND #PWR013
 U 1 1 5F1F77AB
-P 4200 1250
+P 4050 1500
 AR Path="/5F1EB180/5F1F77AB" Ref="#PWR013"  Part="1"
 AR Path="/5F22BCD9/5F22EBB8/5F1F77AB" Ref="#PWR?"  Part="1"
-F 0 "#PWR013" H 4200 1000 50  0001 C CNN
-F 1 "GND" H 4205 1077 50  0000 C CNN
-F 2 "" H 4200 1250 50  0001 C CNN
-F 3 "" H 4200 1250 50  0001 C CNN
-	1    4200 1250
-	-1   0    0    1
+F 0 "#PWR013" H 4050 1250 50  0001 C CNN
+F 1 "GND" H 4055 1327 50  0000 C CNN
+F 2 "" H 4050 1500 50  0001 C CNN
+F 3 "" H 4050 1500 50  0001 C CNN
+	1    4050 1500
+	1    0    0    -1
 $EndComp
 $Comp
@@
 $EndComp
 Wire Wire Line
-	3950 1450 4200 1450
-Connection ~ 4200 1450
+	3950 1450 4050 1450
 Wire Wire Line
 	4200 1450 4200 1850
@@
 Wire Wire Line
 	7700 4250 7700 4600
+$Comp
+L Device:R R?
+U 1 1 5F1FFA0A
+P 5450 2050
+AR Path="/5F115F8B/5F1FFA0A" Ref="R?"  Part="1"
+AR Path="/5F1EB180/5F1FFA0A" Ref="R15"  Part="1"
+AR Path="/5F22BCD9/5F22EBB8/5F1FFA0A" Ref="R?"  Part="1"
+F 0 "R15" H 5450 2200 50  0000 L CNN
+F 1 "R" V 5450 2000 50  0000 L CNN
+F 2 "Resistor_SMD:R_0603_1608Metric_Pad1.05x0.95mm_HandSolder" V 5380 2050 50  0001 C CNN
+F 3 "~" H 5450 2050 50  0001 C CNN
+	1    5450 2050
+	1    0    0    -1
+$EndComp
+$Comp
+L Device:R R?
+U 1 1 5F1FFA16
+P 5450 1650
+AR Path="/5F115F8B/5F1FFA16" Ref="R?"  Part="1"
+AR Path="/5F1EB180/5F1FFA16" Ref="R14"  Part="1"
+AR Path="/5F22BCD9/5F22EBB8/5F1FFA16" Ref="R?"  Part="1"
+F 0 "R14" H 5450 1800 50  0000 L CNN
+F 1 "R" V 5450 1600 50  0000 L CNN
+F 2 "Resistor_SMD:R_0603_1608Metric_Pad1.05x0.95mm_HandSolder" V 5380 1650 50  0001 C CNN
+F 3 "~" H 5450 1650 50  0001 C CNN
+	1    5450 1650
+	1    0    0    -1
+$EndComp
+$Comp
+L Device:R R?
+U 1 1 5F1FFA04
+P 5200 2050
+AR Path="/5F115F8B/5F1FFA04" Ref="R?"  Part="1"
+AR Path="/5F1EB180/5F1FFA04" Ref="R12"  Part="1"
+AR Path="/5F22BCD9/5F22EBB8/5F1FFA04" Ref="R?"  Part="1"
+F 0 "R12" H 5200 2200 50  0000 L CNN
+F 1 "R" V 5200 2000 50  0000 L CNN
+F 2 "Resistor_SMD:R_0603_1608Metric_Pad1.05x0.95mm_HandSolder" V 5130 2050 50  0001 C CNN
+F 3 "~" H 5200 2050 50  0001 C CNN
+	1    5200 2050
+	1    0    0    -1
+$EndComp
+$Comp
+L Device:R R?
+U 1 1 5F1FFA10
+P 5200 1650
+AR Path="/5F115F8B/5F1FFA10" Ref="R?"  Part="1"
+AR Path="/5F1EB180/5F1FFA10" Ref="R11"  Part="1"
+AR Path="/5F22BCD9/5F22EBB8/5F1FFA10" Ref="R?"  Part="1"
+F 0 "R11" H 5200 1800 50  0000 L CNN
+F 1 "R" V 5200 1600 50  0000 L CNN
+F 2 "Resistor_SMD:R_0603_1608Metric_Pad1.05x0.95mm_HandSolder" V 5130 1650 50  0001 C CNN
+F 3 "~" H 5200 1650 50  0001 C CNN
+	1    5200 1650
+	1    0    0    -1
+$EndComp
+$Comp
+L Device:R R?
+U 1 1 5F1FFA23
+P 5000 2050
+AR Path="/5F115F8B/5F1FFA23" Ref="R?"  Part="1"
+AR Path="/5F1EB180/5F1FFA23" Ref="R9"  Part="1"
+AR Path="/5F22BCD9/5F22EBB8/5F1FFA23" Ref="R?"  Part="1"
+F 0 "R9" H 5000 2200 50  0000 L CNN
+F 1 "R" V 5000 2000 50  0000 L CNN
+F 2 "Resistor_SMD:R_0603_1608Metric_Pad1.05x0.95mm_HandSolder" V 4930 2050 50  0001 C CNN
+F 3 "~" H 5000 2050 50  0001 C CNN
+	1    5000 2050
+	1    0    0    -1
+$EndComp
+$Comp
+L Device:R R?
+U 1 1 5F1FFA29
+P 5000 1650
+AR Path="/5F115F8B/5F1FFA29" Ref="R?"  Part="1"
+AR Path="/5F1EB180/5F1FFA29" Ref="R8"  Part="1"
+AR Path="/5F22BCD9/5F22EBB8/5F1FFA29" Ref="R?"  Part="1"
+F 0 "R8" H 4850 1800 50  0000 L CNN
+F 1 "R" V 5000 1600 50  0000 L CNN
+F 2 "Resistor_SMD:R_0603_1608Metric_Pad1.05x0.95mm_HandSolder" V 4930 1650 50  0001 C CNN
+F 3 "~" H 5000 1650 50  0001 C CNN
+	1    5000 1650
+	1    0    0    -1
+$EndComp
+Wire Wire Line
+	5850 1350 5850 2100
+Wire Wire Line
+	5450 1350 5850 1350
+Connection ~ 5450 1350
+Wire Wire Line
+	4050 1500 4050 1450
+Connection ~ 4050 1450
+Wire Wire Line
+	4050 1450 4200 1450
 $EndSCHEMATC
