File: Peltier_V2.sch (KiCad schematic (older format))
At the start: 45 parts, among them U2 MAX1978, U3 DAC081C085, U4 ADC101C021CIMM, U5 REF3333

Commit message: LED_V2
Parts:
- removed C15, C19, C20: 1uF, Capacitor_SMD:C_0805_2012Metric_Pad1.15x1.40mm_HandSolder, symbol Device:C
- removed U3: DAC081C085, Package_SO:VSSOP-8_3.0x3.0mm_P0.65mm, symbol DAC081C085:DAC081C085
- removed U4: ADC101C021CIMM, Package_SO:MSOP-8_3x3mm_P0.65mm, symbol Analog_ADC:ADC101C021CIMM
- removed U5: REF3333, Package_TO_SOT_SMD:SOT-23, symbol REF3333:REF3333
- added C14: 100nF, Capacitor_SMD:C_0603_1608Metric_Pad1.05x0.95mm_HandSolder, symbol Device:C
- added R18, R19, R24, R25, R26, R27, R28, R29: 0R, Resistor_SMD:R_0402_1005Metric, symbol Device:R
- added R30: 10k, Resistor_SMD:R_0603_1608Metric_Pad1.05x0.95mm_HandSolder, symbol Device:R
- added TP1: TestPoint, TestPoint:TestPoint_Pad_D3.0mm, symbol Connector:TestPoint
- added U3: LTC2606IDD, Package_DFN_QFN:DFN-10-1EP_3x3mm_P0.5mm_EP1.65x2.38mm_ThermalVias, symbol DAC:LTC2606IDD
- added U4: ADC121C021CIMM, Package_SO:MSOP-8_3x3mm_P0.65mm, symbol Analog_ADC:ADC121C021CIMM
- C11: value .47uF -> 470nF
- C8: value .047uF -> 47nF
- R20: renamed from R27; footprint Resistor_SMD:R_0603_1608Metric_Pad1.05x0.95mm_HandSolder -> Resistor_SMD:R_0402_1005Metric
- R21: renamed from R28; footprint Resistor_SMD:R_0603_1608Metric_Pad1.05x0.95mm_HandSolder -> Resistor_SMD:R_0402_1005Metric
- R22: renamed from R29; footprint Resistor_SMD:R_0603_1608Metric_Pad1.05x0.95mm_HandSolder -> Resistor_SMD:R_0402_1005Metric
- R23: renamed from R30; footprint Resistor_SMD:R_0603_1608Metric_Pad1.05x0.95mm_HandSolder -> Resistor_SMD:R_0402_1005Metric
- U2: footprint Package_DFN_QFN:QFN-48-1EP_7x7mm_P0.5mm_EP5.45x5.45mm -> Package_DFN_QFN:QFN-48-1EP_7x7mm_P0.5mm_EP5.45x5.45mm_ThermalVias
- renumbered C14 to C15, C18 to C16, C22 to C17, R12 to R10, R9 to R11, R13 to R12, R8 to R13, R11 to R14, R14 to R15, R17 to R16, R16 to R17, R10 to R8, R15 to R9
Connections:
- net labels added: (C1), (C2), (C3), (R1), (R2), (R3), +3.3V
- net labels removed: DC_Current_Monitor
- wire segments 198 -> 214
Other:
- note removed: "These two IC follow same \naddressing schematics,\n can be connected together"
- moved on the sheet: C11, C16, C17, C8, C9, NTC1, R10, R11, R12, R13, R14, R15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

Commit message: LED_Test_V1.3
Parts:
- removed C17: 1uF, Capacitor_SMD:C_0805_2012Metric_Pad1.15x1.40mm_HandSolder, symbol Device:C
- added R46, R47: 0R, Resistor_SMD:R_0402_1005Metric, symbol Device:R
Connections:
- net (C2): no longer C8.1, C9.2, U2.14 (INTOUT), U2.45 (CTLI)
- net +3V3: now also C16.1; no longer C16.2
- net GND: now also C16.2; no longer C16.1
- net VIN: now also R46.1; no longer TP1.1, U4.4 (VIN)
- net NTC: now reaches NTC1.1, R16.2, U2.18 (FB-)
- net NTC: now also R47.1
- new net: C8.1, C9.2, U2.14 (INTOUT), U2.45 (CTLI)
- new net: R46.2, R47.2, TP1.1, U4.4 (VIN)
Other:
- moved on the sheet: C11, C16, C8, C9, R12, R7, R8, TP1
