File: LED2.sch (KiCad schematic (older format))
At the start: 15 parts, among them Q1 FDC6330L, Q2 DMN6075S, U6 LTC1669IMS8, U7 AD8603, U8 PAC1931

Commit message: Current PCB
Parts:
- added R21, R22, R23, R24, R25, R26: 0R, Resistor_SMD:R_0603_1608Metric_Pad1.05x0.95mm_HandSolder, symbol Device:R
Connections:
- net +5V: now also R21.2, R23.2, R25.2
- net GND: now also R22.2, R24.2, R26.2; no longer U6.2 (AD1), U6.3 (AD2), U6.6 (AD0)
- new net: R23.1, R24.1, U6.2 (AD1)
- new net: R25.1, R26.1, U6.3 (AD2)
- new net: R21.1, R22.1, U6.6 (AD0)
Changed lines of the file:
@@
 Connection ~ 6550 4700
-Wire Wire Line
-	3000 3750 3000 3900
-Connection ~ 3000 3900
-Wire Wire Line
-	3000 3900 3000 4050
-Wire Wire Line
-	3000 4050 3000 4300
-Wire Wire Line
-	3000 4300 3550 4300
-Connection ~ 3000 4050
-Connection ~ 3550 4300
 Wire Wire Line
 	7550 4750 7500 4750
@@
 Wire Wire Line
 	6950 1650 7150 1650
+$Comp
+L Device:R R21
+U 1 1 5F313664
+P 2950 4850
+AR Path="/5F1574DE/5F313664" Ref="R21"  Part="1"
+AR Path="/5F22BCD9/5F22EBBD/5F313664" Ref="R?"  Part="1"
+F 0 "R21" H 3020 4896 50  0000 L CNN
+F 1 "0R" V 2950 4800 50  0000 L CNN
+F 2 "Resistor_SMD:R_0603_1608Metric_Pad1.05x0.95mm_HandSolder" V 2880 4850 50  0001 C CNN
+F 3 "~" H 2950 4850 50  0001 C CNN
+	1    2950 4850
+	1    0    0    -1
+$EndComp
+$Comp
+L Device:R R22
+U 1 1 5F313C2A
+P 3250 4850
+AR Path="/5F1574DE/5F313C2A" Ref="R22"  Part="1"
+AR Path="/5F22BCD9/5F22EBBD/5F313C2A" Ref="R?"  Part="1"
+F 0 "R22" H 3320 4896 50  0000 L CNN
+F 1 "0R" V 3250 4800 50  0000 L CNN
+F 2 "Resistor_SMD:R_0603_1608Metric_Pad1.05x0.95mm_HandSolder" V 3180 4850 50  0001 C CNN
+F 3 "~" H 3250 4850 50  0001 C CNN
+	1    3250 4850
+	1    0    0    -1
+$EndComp
+$Comp
+L Device:R R23
+U 1 1 5F313F21
+P 3550 4850
+AR Path="/5F1574DE/5F313F21" Ref="R23"  Part="1"
+AR Path="/5F22BCD9/5F22EBBD/5F313F21" Ref="R?"  Part="1"
+F 0 "R23" H 3620 4896 50  0000 L CNN
+F 1 "0R" V 3550 4800 50  0000 L CNN
+F 2 "Resistor_SMD:R_0603_1608Metric_Pad1.05x0.95mm_HandSolder" V 3480 4850 50  0001 C CNN
+F 3 "~" H 3550 4850 50  0001 C CNN
+	1    3550 4850
+	1    0    0    -1
+$EndComp
+$Comp
+L Device:R R24
+U 1 1 5F31407B
+P 3850 4850
+AR Path="/5F1574DE/5F31407B" Ref="R24"  Part="1"
+AR Path="/5F22BCD9/5F22EBBD/5F31407B" Ref="R?"  Part="1"
+F 0 "R24" H 3920 4896 50  0000 L CNN
+F 1 "0R" V 3850 4800 50  0000 L CNN
+F 2 "Resistor_SMD:R_0603_1608Metric_Pad1.05x0.95mm_HandSolder" V 3780 4850 50  0001 C CNN
+F 3 "~" H 3850 4850 50  0001 C CNN
+	1    3850 4850
+	1    0    0    -1
+$EndComp
+$Comp
+L Device:R R25
+U 1 1 5F314371
+P 4150 4850
+AR Path="/5F1574DE/5F314371" Ref="R25"  Part="1"
+AR Path="/5F22BCD9/5F22EBBD/5F314371" Ref="R?"  Part="1"
+F 0 "R25" H 4220 4896 50  0000 L CNN
+F 1 "0R" V 4150 4800 50  0000 L CNN
+F 2 "Resistor_SMD:R_0603_1608Metric_Pad1.05x0.95mm_HandSolder" V 4080 4850 50  0001 C CNN
+F 3 "~" H 4150 4850 50  0001 C CNN
+	1    4150 4850
+	1    0    0    -1
+$EndComp
+$Comp
+L Device:R R26
+U 1 1 5F314600
+P 4450 4850
+AR Path="/5F1574DE/5F314600" Ref="R26"  Part="1"
+AR Path="/5F22BCD9/5F22EBBD/5F314600" Ref="R?"  Part="1"
+F 0 "R26" H 4520 4896 50  0000 L CNN
+F 1 "0R" V 4450 4800 50  0000 L CNN
+F 2 "Resistor_SMD:R_0603_1608Metric_Pad1.05x0.95mm_HandSolder" V 4380 4850 50  0001 C CNN
+F 3 "~" H 4450 4850 50  0001 C CNN
+	1    4450 4850
+	1    0    0    -1
+$EndComp
+Wire Wire Line
+	2850 3750 3000 3750
+Wire Wire Line
+	2950 4650 2850 4650
+Wire Wire Line
+	2950 4650 2950 4700
+Wire Wire Line
+	2950 4650 3250 4650
+Wire Wire Line
+	3250 4650 3250 4700
+Connection ~ 2950 4650
+$Comp
+L power:GND #PWR034
+U 1 1 5F32073A
+P 3250 5150
+AR Path="/5F1574DE/5F32073A" Ref="#PWR034"  Part="1"
+AR Path="/5F22BCD9/5F22EBBD/5F32073A" Ref="#PWR?"  Part="1"
+F 0 "#PWR034" H 3250 4900 50  0001 C CNN
+F 1 "GND" H 3255 4977 50  0000 C CNN
+F 2 "" H 3250 5150 50  0001 C CNN
+F 3 "" H 3250 5150 50  0001 C CNN
+	1    3250 5150
+	1    0    0    -1
+$EndComp
+Wire Wire Line
+	3250 5000 3250 5100
+Wire Wire Line
+	3850 5000 3850 5100
+Wire Wire Line
+	3850 5100 3250 5100
+Connection ~ 3250 5100
+Wire Wire Line
+	3250 5100 3250 5150
+Wire Wire Line
+	4450 5000 4450 5100
+Wire Wire Line
+	4450 5100 3850 5100
+Connection ~ 3850 5100
+Wire Wire Line
+	3550 4700 3550 4600
+Wire Wire Line
+	3550 4600 3850 4600
+Wire Wire Line
+	3850 4600 3850 4700
+Wire Wire Line
+	2900 3900 3000 3900
+Wire Wire Line
+	2900 4600 3550 4600
+Connection ~ 3550 4600
+Wire Wire Line
+	2950 5000 2950 5450
+$Comp
+L power:+5V #PWR033
+U 1 1 5F332035
+P 2950 5500
+AR Path="/5F1574DE/5F332035" Ref="#PWR033"  Part="1"
+AR Path="/5F22BCD9/5F22EBBD/5F332035" Ref="#PWR?"  Part="1"
+F 0 "#PWR033" H 2950 5350 50  0001 C CNN
+F 1 "+5V" H 2965 5673 50  0000 C CNN
+F 2 "" H 2950 5500 50  0001 C CNN
+F 3 "" H 2950 5500 50  0001 C CNN
+	1    2950 5500
+	-1   0    0    1
+$EndComp
+Wire Wire Line
+	3550 5000 3550 5450
+Wire Wire Line
+	3550 5450 2950 5450
+Wire Wire Line
+	2950 5450 2950 5500
+Connection ~ 2950 5450
+Wire Wire Line
+	2850 3750 2850 4650
+Wire Wire Line
+	2900 3900 2900 4600
+Wire Wire Line
+	4150 5450 3550 5450
+Wire Wire Line
+	4150 5000 4150 5450
+Connection ~ 3550 5450
+Wire Wire Line
+	3000 4050 3000 4500
+Wire Wire Line
+	3000 4500 4150 4500
+Wire Wire Line
+	4450 4500 4450 4700
+Wire Wire Line
+	4150 4700 4150 4500
+Connection ~ 4150 4500
+Wire Wire Line
+	4150 4500 4450 4500
 $EndSCHEMATC

Commit message: Current PCB
Parts:
- removed C18: 100uF, Capacitor_Tantalum_SMD:CP_EIA-7343-15_Kemet-W_Pad2.25x2.55mm_HandSolder, symbol Device:CP
- added C_PWR3, C_PWR4: 100nF, Capacitor_SMD:C_0603_1608Metric_Pad1.05x0.95mm_HandSolder, symbol Device:C
Connections:
- net +5V: now also C_PWR3.2, C_PWR4.1
- net GND: now also C_PWR3.1, C_PWR4.2
Changed lines of the file:
@@
 $EndComp
 Wire Wire Line
-	5100 3350 5100 3050
+	5100 3350 5100 3250
 $Comp
 L LTC1669CMS8:LTC1669CMS8 U6
@@
 	0    -1   -1   0
 $EndComp
-$Comp
-L power:GND #PWR027
-U 1 1 5F1D8B67
-P 6550 4850
-AR Path="/5F1574DE/5F1D8B67" Ref="#PWR027"  Part="1"
-AR Path="/5F22BCD9/5F22EBBD/5F1D8B67" Ref="#PWR?"  Part="1"
-F 0 "#PWR027" H 6550 4600 50  0001 C CNN
-F 1 "GND" H 6555 4677 50  0000 C CNN
-F 2 "" H 6550 4850 50  0001 C CNN
-F 3 "" H 6550 4850 50  0001 C CNN
-	1    6550 4850
-	1    0    0    -1
-$EndComp
 Wire Wire Line
 	6550 4850 6550 4700
@@
 Wire Wire Line
 	6550 1650 6550 2900
-$Comp
-L power:GND #PWR028
-U 1 1 5F1EFE78
-P 7150 1650
-AR Path="/5F1574DE/5F1EFE78" Ref="#PWR028"  Part="1"
-AR Path="/5F22BCD9/5F22EBBD/5F1EFE78" Ref="#PWR?"  Part="1"
-F 0 "#PWR028" H 7150 1400 50  0001 C CNN
-F 1 "GND" V 7155 1522 50  0000 R CNN
-F 2 "" H 7150 1650 50  0001 C CNN
-F 3 "" H 7150 1650 50  0001 C CNN
-	1    7150 1650
-	0    -1   -1   0
-$EndComp
-$Comp
-L Device:CP C18
-U 1 1 5F1EFE7F
-P 6800 1650
-AR Path="/5F1574DE/5F1EFE7F" Ref="C18"  Part="1"
-AR Path="/5F22BCD9/5F22EBBD/5F1EFE7F" Ref="C?"  Part="1"
-F 0 "C18" V 7055 1650 50  0000 C CNN
-F 1 "100uF" V 6964 1650 50  0000 C CNN
-F 2 "Capacitor_Tantalum_SMD:CP_EIA-7343-15_Kemet-W_Pad2.25x2.55mm_HandSolder" H 6838 1500 50  0001 C CNN
-F 3 "~" H 6800 1650 50  0001 C CNN
-	1    6800 1650
-	0    -1   -1   0
-$EndComp
-Wire Wire Line
-	6650 1650 6550 1650
-Connection ~ 6550 1650
-Wire Wire Line
-	6950 1650 7150 1650
 $Comp
 L Device:R R21
@@
 Wire Wire Line
 	4150 4500 4450 4500
+$Comp
+L power:GND #PWR0101
+U 1 1 5F323768
+P 6550 4850
+F 0 "#PWR0101" H 6550 4600 50  0001 C CNN
+F 1 "GND" H 6555 4677 50  0000 C CNN
+F 2 "" H 6550 4850 50  0001 C CNN
+F 3 "" H 6550 4850 50  0001 C CNN
+	1    6550 4850
+	1    0    0    -1
+$EndComp
+$Comp
+L Device:C C_PWR?
+U 1 1 5F33FBAA
+P 3550 2900
+AR Path="/5F0387D4/5F33FBAA" Ref="C_PWR?"  Part="1"
+AR Path="/5F0E5FE6/5F33FBAA" Ref="C_PWR?"  Part="1"
+AR Path="/5F0ECDE4/5F33FBAA" Ref="C_PWR?"  Part="1"
+AR Path="/5F0ED602/5F33FBAA" Ref="C_PWR?"  Part="1"
+AR Path="/5F0EDA8E/5F33FBAA" Ref="C_PWR?"  Part="1"
+AR Path="/5F0EDDEA/5F33FBAA" Ref="C_PWR?"  Part="1"
+AR Path="/5F0EE1DE/5F33FBAA" Ref="C_PWR?"  Part="1"
+AR Path="/5F0EE56E/5F33FBAA" Ref="C_PWR?"  Part="1"
+AR Path="/5F0EE896/5F33FBAA" Ref="C_PWR?"  Part="1"
+AR Path="/5F1BDA41/5F33FBAA" Ref="C_PWR?"  Part="1"
+AR Path="/5F1574DE/5F33FBAA" Ref="C_PWR3"  Part="1"
+AR Path="/5F22BCD9/5F22EBBD/5F33FBAA" Ref="C_PWR?"  Part="1"
+F 0 "C_PWR3" H 3550 3000 39  0000 L CNN
+F 1 "100nF" H 3550 2800 50  0000 L CNN
+F 2 "Capacitor_SMD:C_0603_1608Metric_Pad1.05x0.95mm_HandSolder" H 3588 2750 50  0001 C CNN
+F 3 "~" H 3550 2900 50  0001 C CNN
+	1    3550 2900
+	1    0    0    -1
+$EndComp
+Connection ~ 3550 3050
+Wire Wire Line
+	3550 2700 3550 2750
+$Comp
+L power:GND #PWR037
+U 1 1 5F345D99
+P 3550 2700
+AR Path="/5F1574DE/5F345D99" Ref="#PWR037"  Part="1"
+AR Path="/5F22BCD9/5F22EBBD/5F345D99" Ref="#PWR?"  Part="1"
+F 0 "#PWR037" H 3550 2450 50  0001 C CNN
+F 1 "GND" H 3555 2527 50  0000 C CNN
+F 2 "" H 3550 2700 50  0001 C CNN
+F 3 "" H 3550 2700 50  0001 C CNN
+	1    3550 2700
+	-1   0    0    1
+$EndComp
+$Comp
+L Device:C C_PWR?
+U 1 1 5F346817
+P 5250 3250
+AR Path="/5F0387D4/5F346817" Ref="C_PWR?"  Part="1"
+AR Path="/5F0E5FE6/5F346817" Ref="C_PWR?"  Part="1"
+AR Path="/5F0ECDE4/5F346817" Ref="C_PWR?"  Part="1"
+AR Path="/5F0ED602/5F346817" Ref="C_PWR?"  Part="1"
+AR Path="/5F0EDA8E/5F346817" Ref="C_PWR?"  Part="1"
+AR Path="/5F0EDDEA/5F346817" Ref="C_PWR?"  Part="1"
+AR Path="/5F0EE1DE/5F346817" Ref="C_PWR?"  Part="1"
+AR Path="/5F0EE56E/5F346817" Ref="C_PWR?"  Part="1"
+AR Path="/5F0EE896/5F346817" Ref="C_PWR?"  Part="1"
+AR Path="/5F1BDA41/5F346817" Ref="C_PWR?"  Part="1"
+AR Path="/5F1574DE/5F346817" Ref="C_PWR4"  Part="1"
+AR Path="/5F22BCD9/5F22EBBD/5F346817" Ref="C_PWR?"  Part="1"
+F 0 "C_PWR4" H 5250 3350 39  0000 L CNN
+F 1 "100nF" H 5250 3150 50  0000 L CNN
+F 2 "Capacitor_SMD:C_0603_1608Metric_Pad1.05x0.95mm_HandSolder" H 5288 3100 50  0001 C CNN
+F 3 "~" H 5250 3250 50  0001 C CNN
+	1    5250 3250
+	0    -1   -1   0
+$EndComp
+Connection ~ 5100 3250
+Wire Wire Line
+	5100 3250 5100 3050
+Wire Wire Line
+	5400 3250 5500 3250
+Wire Wire Line
+	5500 3250 5500 2650
+Wire Wire Line
+	5500 2650 5650 2650
+Connection ~ 5650 2650
 $EndSCHEMATC

Commit message: Current PCB
Parts:
- added Extra_FP1: LED, Connector_PinHeader_2.00mm:PinHeader_1x02_P2.00mm_Vertical, symbol Device:LED
- renumbered C_PWR3 to C21, C_PWR4 to C23, C_PWR1 to C24, C_PWR2 to C25
Connections:
- net at D1.1 (K), Q2.3 (D): now also Extra_FP1.1 (K)
- net at D1.2 (A), Q1.2 (D2), Q1.3 (D2): now also Extra_FP1.2 (A)
Changed lines of the file:
@@
 AR Path="/5F0EE896/5F1578A7" Ref="C_PWR?"  Part="1"
 AR Path="/5F1BDA41/5F1578A7" Ref="C_PWR?"  Part="1"
-AR Path="/5F1574DE/5F1578A7" Ref="C_PWR2"  Part="1"
+AR Path="/5F1574DE/5F1578A7" Ref="C25"  Part="1"
 AR Path="/5F22BCD9/5F22EBBD/5F1578A7" Ref="C_PWR?"  Part="1"
-F 0 "C_PWR2" H 8000 3600 50  0000 L CNN
+F 0 "C25" H 8000 3600 50  0000 L CNN
 F 1 "100nF" H 8000 3400 50  0000 L CNN
 F 2 "Capacitor_SMD:C_0603_1608Metric_Pad1.05x0.95mm_HandSolder" H 8038 3350 50  0001 C CNN
@@
 L power:GND #PWR?
 U 1 1 5F1578BA
-P 7850 3150
+P 7700 2950
 AR Path="/5F0387D4/5F1578BA" Ref="#PWR?"  Part="1"
 AR Path="/5F0E5FE6/5F1578BA" Ref="#PWR?"  Part="1"
@@
 AR Path="/5F1574DE/5F1578BA" Ref="#PWR031"  Part="1"
 AR Path="/5F22BCD9/5F22EBBD/5F1578BA" Ref="#PWR?"  Part="1"
-F 0 "#PWR031" H 7850 2900 50  0001 C CNN
-F 1 "GND" H 7850 3000 50  0000 C CNN
-F 2 "" H 7850 3150 50  0001 C CNN
-F 3 "" H 7850 3150 50  0001 C CNN
-	1    7850 3150
-	-1   0    0    1
+F 0 "#PWR031" H 7700 2700 50  0001 C CNN
+F 1 "GND" H 7700 2800 50  0000 C CNN
+F 2 "" H 7700 2950 50  0001 C CNN
+F 3 "" H 7700 2950 50  0001 C CNN
+	1    7700 2950
+	1    0    0    -1
 $EndComp
 $Comp
@@
 AR Path="/5F0EE896/5F1578C7" Ref="C_PWR?"  Part="1"
 AR Path="/5F1BDA41/5F1578C7" Ref="C_PWR?"  Part="1"
-AR Path="/5F1574DE/5F1578C7" Ref="C_PWR1"  Part="1"
+AR Path="/5F1574DE/5F1578C7" Ref="C24"  Part="1"
 AR Path="/5F22BCD9/5F22EBBD/5F1578C7" Ref="C_PWR?"  Part="1"
-F 0 "C_PWR1" H 7650 3600 39  0000 L CNN
+F 0 "C24" H 7650 3600 39  0000 L CNN
 F 1 "100nF" H 7650 3400 50  0000 L CNN
 F 2 "Capacitor_SMD:C_0603_1608Metric_Pad1.05x0.95mm_HandSolder" H 7688 3350 50  0001 C CNN
@@
 $EndComp
 Wire Wire Line
-	6550 3200 6550 3450
+	6550 3200 6550 3300
 Wire Wire Line
 	5500 3650 6000 3650
@@
 F 3 "" H 6300 1200 50  0001 C CNN
 	1    6300 1200
-	0    -1   -1   0
+	1    0    0    -1
 $EndComp
 Wire Wire Line
@@
 L power:GND #PWR025
 U 1 1 5F1C9EAD
-P 5650 2650
+P 5650 2700
 AR Path="/5F1574DE/5F1C9EAD" Ref="#PWR025"  Part="1"
 AR Path="/5F22BCD9/5F22EBBD/5F1C9EAD" Ref="#PWR?"  Part="1"
-F 0 "#PWR025" H 5650 2400 50  0001 C CNN
-F 1 "GND" V 5655 2522 50  0000 R CNN
-F 2 "" H 5650 2650 50  0001 C CNN
-F 3 "" H 5650 2650 50  0001 C CNN
-	1    5650 2650
+F 0 "#PWR025" H 5650 2450 50  0001 C CNN
+F 1 "GND" V 5655 2572 50  0000 R CNN
+F 2 "" H 5650 2700 50  0001 C CNN
+F 3 "" H 5650 2700 50  0001 C CNN
+	1    5650 2700
 	1    0    0    -1
 $EndComp
@@
 AR Path="/5F0EE896/5F33FBAA" Ref="C_PWR?"  Part="1"
 AR Path="/5F1BDA41/5F33FBAA" Ref="C_PWR?"  Part="1"
-AR Path="/5F1574DE/5F33FBAA" Ref="C_PWR3"  Part="1"
+AR Path="/5F1574DE/5F33FBAA" Ref="C21"  Part="1"
 AR Path="/5F22BCD9/5F22EBBD/5F33FBAA" Ref="C_PWR?"  Part="1"
-F 0 "C_PWR3" H 3550 3000 39  0000 L CNN
+F 0 "C21" H 3550 3000 39  0000 L CNN
 F 1 "100nF" H 3550 2800 50  0000 L CNN
 F 2 "Capacitor_SMD:C_0603_1608Metric_Pad1.05x0.95mm_HandSolder" H 3588 2750 50  0001 C CNN
@@
 L power:GND #PWR037
 U 1 1 5F345D99
-P 3550 2700
+P 3350 2700
 AR Path="/5F1574DE/5F345D99" Ref="#PWR037"  Part="1"
 AR Path="/5F22BCD9/5F22EBBD/5F345D99" Ref="#PWR?"  Part="1"
-F 0 "#PWR037" H 3550 2450 50  0001 C CNN
-F 1 "GND" H 3555 2527 50  0000 C CNN
-F 2 "" H 3550 2700 50  0001 C CNN
-F 3 "" H 3550 2700 50  0001 C CNN
-	1    3550 2700
-	-1   0    0    1
+F 0 "#PWR037" H 3350 2450 50  0001 C CNN
+F 1 "GND" H 3355 2527 50  0000 C CNN
+F 2 "" H 3350 2700 50  0001 C CNN
+F 3 "" H 3350 2700 50  0001 C CNN
+	1    3350 2700
+	1    0    0    -1
 $EndComp
 $Comp
@@
 AR Path="/5F0EE896/5F346817" Ref="C_PWR?"  Part="1"
 AR Path="/5F1BDA41/5F346817" Ref="C_PWR?"  Part="1"
-AR Path="/5F1574DE/5F346817" Ref="C_PWR4"  Part="1"
+AR Path="/5F1574DE/5F346817" Ref="C23"  Part="1"
 AR Path="/5F22BCD9/5F22EBBD/5F346817" Ref="C_PWR?"  Part="1"
-F 0 "C_PWR4" H 5250 3350 39  0000 L CNN
+F 0 "C23" H 5250 3350 39  0000 L CNN
 F 1 "100nF" H 5250 3150 50  0000 L CNN
 F 2 "Capacitor_SMD:C_0603_1608Metric_Pad1.05x0.95mm_HandSolder" H 5288 3100 50  0001 C CNN
@@
 	5500 2650 5650 2650
 Connection ~ 5650 2650
+$Comp
+L Device:LED Extra_FP1
+U 1 1 5F3C2DB0
+P 6200 3050
+AR Path="/5F1574DE/5F3C2DB0" Ref="Extra_FP1"  Part="1"
+AR Path="/5F22BCD9/5F22EBBD/5F3C2DB0" Ref="D?"  Part="1"
+F 0 "Extra_FP1" H 6400 3150 50  0000 R CNN
+F 1 "LED" V 6148 2932 50  0000 R CNN
+F 2 "Connector_PinHeader_2.00mm:PinHeader_1x02_P2.00mm_Vertical" H 6200 3050 50  0001 C CNN
+F 3 "~" H 6200 3050 50  0001 C CNN
+	1    6200 3050
+	0    -1   -1   0
+$EndComp
+Wire Wire Line
+	6200 2900 6550 2900
+Connection ~ 6550 2900
+Wire Wire Line
+	6200 3200 6200 3300
+Wire Wire Line
+	6200 3300 6550 3300
+Connection ~ 6550 3300
+Wire Wire Line
+	6550 3300 6550 3450
+Wire Wire Line
+	3350 2700 3550 2700
+Wire Wire Line
+	7850 3150 7850 2950
+Wire Wire Line
+	7850 2950 7700 2950
+Wire Wire Line
+	5650 2700 5650 2650
 $EndSCHEMATC

Commit message: LED_V2
Parts:
- removed C17: .1uF, Capacitor_SMD:C_0805_2012Metric_Pad1.15x1.40mm_HandSolder, symbol Device:C
- removed Extra_FP1: LED, Connector_PinHeader_2.00mm:PinHeader_1x02_P2.00mm_Vertical, symbol Device:LED
- removed U6: LTC1669IMS8, Package_SO:MSOP-8_3x3mm_P0.65mm, symbol LTC1669CMS8:LTC1669CMS8
- removed U8: PAC1931, Package_DFN_QFN:UQFN-16-1EP_4x4mm_P0.65mm_EP2.7x2.7mm, symbol LED_test-rescue:PAC1931-PAC1931-LED_test-rescue
- added D2: LED, LED_THT:LED_D3.0mm, symbol Device:LED
- added NT1: Net-Tie_2, NetTie:NetTie-2_SMD_Pad0.5mm, symbol Device:Net-Tie_2
- added R33, R36, R40, R42: 0, Resistor_SMD:R_0402_1005Metric, symbol Device:R
- added R34, R37: 0R, Resistor_SMD:R_0402_1005Metric, symbol Device:R
- added U5: LTC2606IDD, Package_DFN_QFN:DFN-10-1EP_3x3mm_P0.5mm_EP1.65x2.38mm_ThermalVias, symbol DAC:LTC2606IDD
- added U7: PAC1932, Package_DFN_QFN:QFN-16-1EP_4x4mm_P0.65mm_EP2.5x2.5mm_ThermalVias, symbol PAC1931:PAC1932
- added U8: REF3333, Package_TO_SOT_SMD:SOT-23, symbol REF3333:REF3333
- D1: footprint LED_pad:LED_PAD -> LED_THT:LED_D3.0mm
- R31: renamed from R21; footprint Resistor_SMD:R_0603_1608Metric_Pad1.05x0.95mm_HandSolder -> Resistor_SMD:R_0402_1005Metric
- R32: renamed from R22; footprint Resistor_SMD:R_0603_1608Metric_Pad1.05x0.95mm_HandSolder -> Resistor_SMD:R_0402_1005Metric
- R35: renamed from R23; footprint Resistor_SMD:R_0603_1608Metric_Pad1.05x0.95mm_HandSolder -> Resistor_SMD:R_0402_1005Metric
- R38: renamed from R24; footprint Resistor_SMD:R_0603_1608Metric_Pad1.05x0.95mm_HandSolder -> Resistor_SMD:R_0402_1005Metric
- R39: renamed from R25; footprint Resistor_SMD:R_0603_1608Metric_Pad1.05x0.95mm_HandSolder -> Resistor_SMD:R_0402_1005Metric
- R41: renamed from R26; footprint Resistor_SMD:R_0603_1608Metric_Pad1.05x0.95mm_HandSolder -> Resistor_SMD:R_0402_1005Metric
- renumbered C21 to C18, C23 to C19, C16 to C20, C24 to C21, C25 to C22, R18 to R43, R19 to R44, R20 to R45, U7 to U6
Connections:
- net +12V: now also R42.1
- net +3V3: now also U7.1 (SLOW/ALERT), U7.15 (VDD_I/O), U7.16 (PWRDN)
- net +5V: now also R34.2, R36.1, R40.1, U5.9 (VCC), U7.2 (VDD), U8.1 (IN); no longer C19.1, U6.5 (V+)
- net GND: now also NT1.2, R37.2, U5.11 (EP), U5.8 (GND), U7.10 (SENSE4+), U7.3 (GND), U7.7 (SENSE3-), U7.8 (SENSE3+), U7.9 (SENSE4-), U8.3 (GND); no longer R45.2
- net SM_CLK: now also U5.3 (SCL), U7.4 (SM_CLK)
- net SM_DATA: now also U5.2 (SDA), U7.5 (SM_DATA)
- net at R45.1, U6.4 (-): now also D2.1 (K), U7.13 (SENSE2+); no longer Q2.2 (S)
- net at R_Address1.1: now also U7.6 (ADDRSEL_)
- net at U6.3 (+): now also U5.7 (Vout)
- net at R35.1, R38.1: now also U5.5 (CA1)
- net at R39.1, R41.1: now also U5.1 (CA2)
- net at R31.1, R32.1: now also U5.4 (CA0)
- new net: C19.1, R40.2, R42.2, U6.5 (V+)
- new net: NT1.1, R45.2, U7.14 (SENSE2-)
- new net: D2.2 (A), Q2.2 (S), U7.11 (SENSE1+), U7.12 (SENSE1-)
- new net: R34.1, R37.1, U5.10 (LDAC)
- new net: R33.2, R36.2, U5.6 (REF)
- new net: R33.1, U8.2 (OUT)
Other:
- moved on the sheet: C18, R45

Commit message: LED_Test_V1.3
Parts:
- added R48: 100k, Resistor_SMD:R_0603_1608Metric_Pad1.05x0.95mm_HandSolder, symbol Device:R
- R45: footprint Resistor_SMD:R_0603_1608Metric_Pad1.05x0.95mm_HandSolder -> Resistor_SMD:R_1206_3216Metric_Pad1.42x1.75mm_HandSolder
Connections:
- net GND: now also R48.2
- net LED_Power: now also R48.1
Changed lines of the file:
@@
 F 0 "R45" H 6620 4746 50  0000 L CNN
 F 1 ".1" V 6550 4650 50  0000 L CNN
-F 2 "Resistor_SMD:R_0603_1608Metric_Pad1.05x0.95mm_HandSolder" V 6480 4700 50  0001 C CNN
+F 2 "Resistor_SMD:R_1206_3216Metric_Pad1.42x1.75mm_HandSolder" V 6480 4700 50  0001 C CNN
 F 3 "~" H 6550 4700 50  0001 C CNN
 	1    6550 4700
@@
 $EndComp
 Wire Wire Line
-	5150 2050 5600 2050
+	5150 2050 5500 2050
 Wire Wire Line
 	5600 750  5600 1200
@@
 AR Path="/5F0EE896/5FE062F2" Ref="#PWR?"  Part="1"
 AR Path="/5F1BDA41/5FE062F2" Ref="#PWR?"  Part="1"
-AR Path="/5F1574DE/5FE062F2" Ref="#PWR?"  Part="1"
+AR Path="/5F1574DE/5FE062F2" Ref="#PWR056"  Part="1"
 AR Path="/5F22BCD9/5F22EBBD/5FE062F2" Ref="#PWR?"  Part="1"
-F 0 "#PWR?" H 6750 5150 50  0001 C CNN
+F 0 "#PWR056" H 6750 5150 50  0001 C CNN
 F 1 "GND" H 6755 5227 50  0000 C CNN
 F 2 "" H 6750 5400 50  0001 C CNN
@@
 Wire Wire Line
 	6550 5400 6550 5450
+$Comp
+L Device:R R_Address?
+U 1 1 5FF80A53
+P 5500 2300
+AR Path="/5F0387D4/5FF80A53" Ref="R_Address?"  Part="1"
+AR Path="/5F0E5FE6/5FF80A53" Ref="R_Address?"  Part="1"
+AR Path="/5F0ECDE4/5FF80A53" Ref="R_Address?"  Part="1"
+AR Path="/5F0ED602/5FF80A53" Ref="R_Address?"  Part="1"
+AR Path="/5F0EDA8E/5FF80A53" Ref="R_Address?"  Part="1"
+AR Path="/5F0EDDEA/5FF80A53" Ref="R_Address?"  Part="1"
+AR Path="/5F0EE1DE/5FF80A53" Ref="R_Address?"  Part="1"
+AR Path="/5F0EE56E/5FF80A53" Ref="R_Address?"  Part="1"
+AR Path="/5F0EE896/5FF80A53" Ref="R_Address?"  Part="1"
+AR Path="/5F1BDA41/5FF80A53" Ref="R_Address?"  Part="1"
+AR Path="/5F1574DE/5FF80A53" Ref="R48"  Part="1"
+AR Path="/5F22BCD9/5F22EBBD/5FF80A53" Ref="R_Address?"  Part="1"
+F 0 "R48" H 5350 2250 31  0000 L CNN
+F 1 "100k" V 5500 2200 50  0000 L CNN
+F 2 "Resistor_SMD:R_0603_1608Metric_Pad1.05x0.95mm_HandSolder" V 5430 2300 50  0001 C CNN
+F 3 "~" H 5500 2300 50  0001 C CNN
+	1    5500 2300
+	1    0    0    -1
+$EndComp
+Wire Wire Line
+	5500 2150 5500 2050
+Connection ~ 5500 2050
+Wire Wire Line
+	5500 2050 5600 2050
+Wire Wire Line
+	5500 2450 5500 2650
+Connection ~ 5500 2650
 $EndSCHEMATC

Commit message: LED_Test_Board_V1.3
Parts:
- removed R37: 0R, Resistor_SMD:R_0402_1005Metric, symbol Device:R
- added C17: 100pF, Capacitor_SMD:C_0603_1608Metric_Pad1.05x0.95mm_HandSolder, symbol Device:C
- added C23: 100nF, Capacitor_SMD:C_0603_1608Metric_Pad1.05x0.95mm_HandSolder, symbol Device:C
- added C24: 22pF, Capacitor_SMD:C_0603_1608Metric_Pad1.05x0.95mm_HandSolder, symbol Device:C
- added R49: 100K, Resistor_SMD:R_0603_1608Metric_Pad1.05x0.95mm_HandSolder, symbol Device:R
- added R50: 10K, Resistor_SMD:R_0603_1608Metric_Pad1.05x0.95mm_HandSolder, symbol Device:R
- added TP2, TP3, TP4: TestPoint, TestPoint:TestPoint_Pad_D1.0mm, symbol Connector:TestPoint
- added U9: AD8603, Package_TO_SOT_SMD:TSOT-23-5, symbol Amplifier_Operational:AD8603
- R34: value 0R -> 10K; footprint Resistor_SMD:R_0402_1005Metric -> Resistor_SMD:R_0603_1608Metric_Pad1.05x0.95mm_HandSolder
- R42: value 0 -> 2K; footprint Resistor_SMD:R_0402_1005Metric -> Resistor_SMD:R_0603_1608Metric_Pad1.05x0.95mm_HandSolder
- R43: value 100 -> 10K
- R44: value 1k -> 0; footprint Resistor_SMD:R_0603_1608Metric_Pad1.05x0.95mm_HandSolder -> Resistor_SMD:R_0402_1005Metric
Connections:
- net +12V: no longer R42.1
- net +5V: now also C19.1, U6.5 (V+), C23.1, U9.5 (V+); no longer R34.2, R40.1
- net GND: now also Q1.1 (S1), R42.2, U5.10 (LDAC), C23.2, U9.2 (V-); no longer R44.2, U7.10 (SENSE4+), U7.7 (SENSE3-), U7.8 (SENSE3+), U7.9 (SENSE4-)
- net at Q2.1 (G), U6.1: now also C17.1
- net at U6.3 (+): now also R34.1; no longer U5.7 (Vout)
- net at D2.1 (K), R45.1, U7.13 (SENSE2+): now also R44.1; no longer U6.4 (-)
- net at D1.1 (K), Q2.3 (D): now also U7.11 (SENSE1+), U7.12 (SENSE1-)
- net at D1.2 (A), Q1.2 (D2), Q1.3 (D2): now also U7.7 (SENSE3-), U7.8 (SENSE3+)
- net at D2.2 (A), Q2.2 (S): now also R50.2; no longer U7.11 (SENSE1+), U7.12 (SENSE1-)
- new net: C17.2, R40.2, R44.2, U6.4 (-)
- new net: R34.2, TP2.1, U5.7 (Vout)
- new net: TP4.1, U7.10 (SENSE4+)
- new net: TP3.1, U7.9 (SENSE4-)
- new net: C24.1, R40.1, R42.1, R49.2, U9.1
- new net: R50.1, U9.3 (+)
- new net: C24.2, R49.1, U9.4 (-)
Other:
- moved on the sheet: C18, C19, C20, C21, C22, D1, D2, Q1, Q2, R31, R32, R33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
