File: LED_test_V1.3.kicad_pcb (KiCad board)
At the start: 2 copper layers, 100 x 100 mm, 94 parts, among them J1 Conn_01x08_Male, J2 Conn_01x10_Male, Q1 FDC6330L, Q2 DMN6075S, U1 MAX14662, U2 MAX1978, U3 LTC2606IDD, U4 ADC121C021CIMM, U5 LTC2606IDD, U6 AD8603, U7 PAC1932, U8 REF3333

Commit message: LED_Test_Board_V1.3
Routing:
- net GND: track 87.8 -> 120.9 mm

Commit message: LED_Test_Board_V1.3
Parts:
- removed R37: 0R, Resistor_SMD:R_0402_1005Metric
- added C17: 100pF, Capacitor_SMD:C_0603_1608Metric_Pad1.05x0.95mm_HandSolder, F.Cu at (176.8, 119.0)
- added C23: 100nF, Capacitor_SMD:C_0603_1608Metric_Pad1.05x0.95mm_HandSolder, F.Cu at (179.9, 69.9)
- added C24: 22pF, Capacitor_SMD:C_0603_1608Metric_Pad1.05x0.95mm_HandSolder, F.Cu at (183.6, 66.1)
- added R49: 100K, Resistor_SMD:R_0603_1608Metric_Pad1.05x0.95mm_HandSolder, F.Cu at (183.6, 64.2)
- added R50: 10K, Resistor_SMD:R_0603_1608Metric_Pad1.05x0.95mm_HandSolder, F.Cu at (190.5, 68.9)
- added TP2: TestPoint, TestPoint:TestPoint_Pad_D1.0mm, F.Cu at (173.5, 129.2)
- added TP3: TestPoint, TestPoint:TestPoint_Pad_D1.0mm, F.Cu at (196.6, 127.0)
- added TP4: TestPoint, TestPoint:TestPoint_Pad_D1.0mm, F.Cu at (196.5, 124.8)
- added U9: AD8603, Package_TO_SOT_SMD:TSOT-23-5, F.Cu at (184.1, 69.8)
- R34: value 0R -> 10K; footprint Resistor_SMD:R_0402_1005Metric -> Resistor_SMD:R_0603_1608Metric_Pad1.05x0.95mm_HandSolder
- R42: value 0 -> 2K; footprint Resistor_SMD:R_0402_1005Metric -> Resistor_SMD:R_0603_1608Metric_Pad1.05x0.95mm_HandSolder
- R43: value 100 -> 10K
- R44: value 1k -> 0; footprint Resistor_SMD:R_0603_1608Metric_Pad1.05x0.95mm_HandSolder -> Resistor_SMD:R_0402_1005Metric
- moved R42 48.0 mm to (186.3, 74.2)
- moved NTC1 33.4 mm to (126.8, 61.8)
- moved R16 33.1 mm to (129.6, 61.4)
- moved C5 32.5 mm to (113.4, 61.5)
- moved C10 32.5 mm to (141.1, 67.2)
- moved C11 32.5 mm to (122.2, 76.7)
- moved C12 32.5 mm to (147.7, 81.8)
- moved C13 32.5 mm to (140.3, 56.2)
- moved C15 32.5 mm to (140.3, 85.8)
- moved C2 32.5 mm to (127.2, 82.2)
- moved C3 32.5 mm to (137.4, 76.4)
- moved C4 32.5 mm to (141.1, 69.9)
- moved C7 32.5 mm to (132.8, 63.6)
- moved C8 32.5 mm to (120.1, 69.6)
- moved C9 32.5 mm to (122.1, 66.0)
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Connections:
- C19 pad 1: Net-(C19-Pad1) -> +5V
- Q1 pad 1: Net-(Q1-Pad1) -> GND
- R34 pad 2: +5V -> Net-(R34-Pad2)
- R40 pad 1: +5V -> Net-(C24-Pad1)
- R40 pad 2: Net-(C19-Pad1) -> Net-(C17-Pad2)
- R42 pad 1: +12V -> Net-(C24-Pad1)
- R42 pad 2: Net-(C19-Pad1) -> GND
- R44 pad 1: Net-(Q1-Pad1) -> Net-(D2-Pad1)
- R44 pad 2: GND -> Net-(C17-Pad2)
- U5 pad 10: Net-(R34-Pad1) -> GND
- U5 pad 7: Net-(U5-Pad7) -> Net-(R34-Pad2)
- U6 pad 3: Net-(U5-Pad7) -> Net-(R34-Pad1)
- U6 pad 4: Net-(D2-Pad1) -> Net-(C17-Pad2)
- U6 pad 5: Net-(C19-Pad1) -> +5V
- U7 pad 10: GND -> Net-(TP4-Pad1)
- U7 pad 11: Net-(D2-Pad2) -> Net-(D1-Pad1)
- U7 pad 12: Net-(D2-Pad2) -> Net-(D1-Pad1)
- U7 pad 7: GND -> Net-(D1-Pad2)
- U7 pad 8: GND -> Net-(D1-Pad2)
- U7 pad 9: GND -> Net-(TP3-Pad1)
Routing:
- net Net-(D1-Pad1): track 10.2 -> 80.4 mm
- net Net-(D1-Pad2): track 16.7 -> 78.0 mm, vias 0 -> 1
- net Net-(C24-Pad1): track 0.00 -> 58.5 mm, vias 0 -> 2
- net +5V: track 393.5 -> 415.3 mm
- net Net-(D2-Pad2): track 59.0 -> 37.4 mm, vias 0 -> 1
- net /Sheet5F1EB17F/DATA: track 173.6 -> 155.7 mm
- net /Sheet5F1EB17F/CLOCK: track 173.9 -> 158.0 mm
- net +12V: track 74.9 -> 61.7 mm, vias 2 -> 0
- net Net-(C17-Pad2): track 0.00 -> 11.2 mm
- net Net-(U5-Pad7): track 11.1 -> 0.00 mm
- net Net-(R34-Pad2): track 0.00 -> 10.3 mm
- net Net-(C19-Pad1): track 7.32 -> 0.00 mm
- net Net-(R_Address1-Pad1): track 2.32 -> 9.29 mm
- net Net-(D2-Pad1): track 48.7 -> 55.6 mm
- net Net-(R46-Pad2): track 14.7 -> 8.30 mm
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